File: hardware/sensor-1/sensor-1.kicad_sch (KiCad schematic)
At the start: 15 parts, among them J101 2x05_Horizontal, U101 A31010SEHALT-10, U102 A31010SEHALT-10, U103 A31010SEHALT-10

Commit message: Update sensors
Parts:
- C101, C103, C104: footprint Capacitor_SMD:C_0603_1608Metric -> V2_Capacitor_SMD:C_0603; symbol Device:C_Small -> V2_Device:C_0603_0u1; Manufacturer (none) -> TDK; Mouser (none) -> 810-CGA3E2X7R1H104MA; Product (none) -> CGA3E2X7R1H104M080AA; Rating (none) -> 50V
- FID101, FID102: value Fiducial -> Fiducial_Paste
- INFO101: value ORDER-NUMBER -> Order_Number
- J101: Manufacturer (none) -> Amphenol FCI; Mouser (none) -> 649-200211120001T4LF; Product (none) -> 20021112-00010T4LF
