File: hardware/sax2/PowerSupply.kicad_sch (KiCad schematic)
At the start: 8 parts, among them U1201 TPSM33625

Commit message: Refresh footprints
Parts:
- C1205: Rating (none) -> 50V
Changed lines of the file:
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@@
+			)
+		)
+		(property "Rating" "50V"
+			(at 128.27 130.81 0)
+			(effects
+				(font
+					(size 1.27 1.27)
+				)
+				(hide yes)
 			)
 		)

Commit message: Refresh
Parts:
- C1205: Manufacturer YAGEO -> TDK; Mouser 603-CC603KRX7R9BB105 -> 810-CGA3E3X7R1H105K0; Product CC0603KRX7R9BB105 -> CGA3E3X7R1H105K080AB
Changed lines of the file:
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@@
 			)
 		)
-		(property "Mouser" "603-CC603KRX7R9BB105"
+		(property "Mouser" "810-CGA3E3X7R1H105K0"
 			(at 128.27 128.27 0)
 			(effects
@@
 			)
 		)
-		(property "Product" "CC0603KRX7R9BB105"
+		(property "Product" "CGA3E3X7R1H105K080AB"
 			(at 128.27 125.73 0)
 			(effects
@@
 			)
 		)
-		(property "Manufacturer" "YAGEO"
+		(property "Manufacturer" "TDK"
 			(at 128.27 123.19 0)
 			(effects

Commit message: Update library
Parts:
- C1201: Rating (none) -> 50V; Voltage 50V -> (none)
- C1202: Rating (none) -> 50V
- C1203, C1204: Rating (none) -> 25V; Voltage 25V -> (none)
Changed lines of the file:
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@@
+			)
+		)
+		(property "Rating" "50V"
+			(at 109.22 120.65 0)
+			(effects
+				(font
+					(size 1.27 1.27)
+				)
+				(hide yes)
 			)
 		)
@@
 			)
 		)
-		(property "Voltage" "25V"
-			(at 195.58 118.11 0)
-			(effects
-				(font
-					(size 1.27 1.27)
-				)
-				(hide yes)
-			)
-		)
 		(property "Product" "CGA6P3X7R1E226M250AE"
 			(at 195.58 115.57 0)
@@
 			)
 		)
+		(property "Rating" "25V"
+			(at 195.58 118.11 0)
+			(effects
+				(font
+					(size 1.27 1.27)
+				)
+				(hide yes)
+			)
+		)
 		(pin "1"
 		)
@@
 			)
 		)
-		(property "Description" "Power symbol creates a global label with name \"GND\" , ground"
+		(property "Description" ""
 			(at 185.42 100.33 0)
 			(effects
@@
 			)
 		)
-		(property "Description" "Power symbol creates a global label with name \"GND\" , ground"
+		(property "Description" ""
 			(at 195.58 100.33 0)
 			(effects
@@
 			)
 		)
-		(property "Description" "Power symbol creates a global label with name \"GND\" , ground"
+		(property "Description" ""
 			(at 97.79 100.33 0)
 			(effects
@@
 			)
 		)
-		(property "Description" "Power symbol creates a global label with name \"GND\" , ground"
+		(property "Description" ""
 			(at 172.72 105.41 0)
 			(effects
@@
 			)
 		)
-		(property "Description" "Power symbol creates a global label with name \"GND\" , ground"
+		(property "Description" ""
 			(at 109.22 100.33 0)
 			(effects
@@
 			)
 		)
-		(property "Voltage" "25V"
-			(at 185.42 118.11 0)
-			(effects
-				(font
-					(size 1.27 1.27)
-				)
-				(hide yes)
-			)
-		)
 		(property "Product" "CGA6P3X7R1E226M250AE"
 			(at 185.42 115.57 0)
@@
 			)
 		)
+		(property "Rating" "25V"
+			(at 185.42 118.11 0)
+			(effects
+				(font
+					(size 1.27 1.27)
+				)
+				(hide yes)
+			)
+		)
 		(pin "1"
 		)
@@
 			)
 		)
-		(property "Description" "Power symbol creates a global label with name \"GND\" , ground"
+		(property "Description" ""
 			(at 128.27 110.49 0)
 			(effects
@@
 			)
 		)
-		(property "Description" "Power symbol creates a global label with name \"GND\" , ground"
+		(property "Description" ""
 			(at 148.59 115.57 0)
 			(effects
@@
 			)
 		)
-		(property "Voltage" "50V"
+		(property "Rating" "50V"
 			(at 97.79 118.11 0)
 			(effects

Commit message: Update library
Parts:
- U1201: value TPSM33625 -> TPSM365R6FRDNR; footprint V2_Converter_DCDC:TPSM33625 -> V2_Converter_DCDC:QFN-11; symbol V2_Converter_DCDC:TPSM33625 -> V2_Converter_DCDC:TPSM365R6FRDNR; Mouser 595-TPSM33625RDNR -> 595-TPSM365R6FRDNR; Product TPSM33625RDNR -> TPSM365R6FRDNR; Rating (none) -> 600mA
Changed lines of the file:
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@@
 	)
 	(symbol
-		(lib_id "V2_Converter_DCDC:TPSM33625")
+		(lib_id "V2_Converter_DCDC:TPSM365R6FRDNR")
 		(at 148.59 102.87 0)
 		(unit 1)
@@
 			)
 		)
-		(property "Value" "TPSM33625"
+		(property "Value" "TPSM365R6FRDNR"
 			(at 144.78 90.17 0)
 			(effects
@@
 			)
 		)
-		(property "Footprint" "V2_Converter_DCDC:TPSM33625"
+		(property "Footprint" "V2_Converter_DCDC:QFN-11"
 			(at 148.59 118.11 0)
 			(effects
@@
 			)
 		)
-		(property "Datasheet" "https://www.ti.com/lit/ds/symlink/tpsm33625.pdf"
+		(property "Datasheet" ""
 			(at 153.67 118.11 0)
 			(effects
@@
 			)
 		)
-		(property "Mouser" "595-TPSM33625RDNR"
+		(property "Mouser" "595-TPSM365R6FRDNR"
 			(at 148.59 151.13 0)
 			(effects
@@
 			)
 		)
-		(property "Product" "TPSM33625RDNR"
+		(property "Product" "TPSM365R6FRDNR"
 			(at 148.59 148.59 0)
 			(effects
 				(font
+					(size 1.27 1.27)
+				)
+				(hide yes)
+			)
+		)
+		(property "Rating" "600mA"
+			(at 148.59 153.67 0)
+			(effects
+				(font
