File: hardware/sax2/PowerSupply.kicad_sch (KiCad schematic)
At the start: 8 parts, among them U1201 TPSM365R6FRDNR

Commit message: Update Library
Parts:
- C1201: symbol V2_Device:C_1210_10u -> V2_Capacitor:1210_10u
- C1202: symbol V2_Device:C_0603_0u1 -> V2_Capacitor:0603_0u1
- C1203, C1204: value 22u -> 10u; symbol V2_Device:C_1210_22u -> V2_Capacitor:1210_22u
- C1205: symbol V2_Device:C_0603_1u -> V2_Capacitor:0603_1u
- R1201: symbol V2_Device:R_0603_40k2 -> V2_Resistor:0603_40k2
- R1202: symbol V2_Device:R_0603_10k -> V2_Resistor:0603_10k
Changed lines of the file:
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@@
 	)
 	(symbol
-		(lib_id "V2_Device:C_0603_0u1")
+		(lib_id "V2_Capacitor:0603_0u1")
 		(at 109.22 97.79 0)
 		(unit 1)
@@
 	)
 	(symbol
-		(lib_id "V2_Device:C_1210_22u")
+		(lib_id "V2_Capacitor:1210_22u")
 		(at 195.58 97.79 0)
 		(unit 1)
@@
 			)
 		)
-		(property "Value" "22u"
+		(property "Value" "10u"
 			(at 198.12 99.06 0)
 			(effects
@@
 	)
 	(symbol
-		(lib_id "V2_Device:R_0603_40k2")
+		(lib_id "V2_Resistor:0603_40k2")
 		(at 172.72 97.79 0)
 		(unit 1)
@@
 		(on_board yes)
 		(dnp no)
-		(property "Reference" "#PWR01203"
+		(property "Reference" "#PWR1203"
 			(at 185.42 106.68 0)
 			(effects
@@
 			(project "sax2"
 				(path "/6c8448b4-b04d-47e1-934e-e40cbe27a7be/095cddf1-6522-4d3b-885d-b21acd91d0c6"
-					(reference "#PWR01203")
+					(reference "#PWR1203")
 					(unit 1)
 				)
@@
 		(on_board yes)
 		(dnp no)
-		(property "Reference" "#PWR01204"
+		(property "Reference" "#PWR1204"
 			(at 195.58 106.68 0)
 			(effects
@@
 			(project "sax2"
 				(path "/6c8448b4-b04d-47e1-934e-e40cbe27a7be/095cddf1-6522-4d3b-885d-b21acd91d0c6"
-					(reference "#PWR01204")
+					(reference "#PWR1204")
 					(unit 1)
 				)
@@
 		(on_board yes)
 		(dnp no)
-		(property "Reference" "#PWR01201"
+		(property "Reference" "#PWR1201"
 			(at 97.79 106.68 0)
 			(effects
@@
 			(project "sax2"
 				(path "/6c8448b4-b04d-47e1-934e-e40cbe27a7be/095cddf1-6522-4d3b-885d-b21acd91d0c6"
-					(reference "#PWR01201")
+					(reference "#PWR1201")
 					(unit 1)
 				)
@@
 		(on_board yes)
 		(dnp no)
-		(property "Reference" "#PWR01205"
+		(property "Reference" "#PWR1205"
 			(at 172.72 111.76 0)
 			(effects
@@
 			(project "sax2"
 				(path "/6c8448b4-b04d-47e1-934e-e40cbe27a7be/095cddf1-6522-4d3b-885d-b21acd91d0c6"
-					(reference "#PWR01205")
+					(reference "#PWR1205")
 					(unit 1)
 				)
@@
 		(on_board yes)
 		(dnp no)
-		(property "Reference" "#PWR01202"
+		(property "Reference" "#PWR1202"
 			(at 109.22 106.68 0)
 			(effects
@@
 			(project "sax2"
 				(path "/6c8448b4-b04d-47e1-934e-e40cbe27a7be/095cddf1-6522-4d3b-885d-b21acd91d0c6"
-					(reference "#PWR01202")
-					(unit 1)
-				)
-			)
-		)
-	)
-	(symbol
-		(lib_id "V2_Device:C_0603_1u")
+					(reference "#PWR1202")
+					(unit 1)
+				)
+			)
+		)
+	)
+	(symbol
+		(lib_id "V2_Capacitor:0603_1u")
 		(at 128.27 107.95 0)
 		(unit 1)
@@
 	)
 	(symbol
-		(lib_id "V2_Device:C_1210_22u")
+		(lib_id "V2_Capacitor:1210_22u")
 		(at 185.42 97.79 0)
 		(unit 1)
@@
 			)
 		)
-		(property "Value" "22u"
+		(property "Value" "10u"
 			(at 187.96 98.806 0)
 			(effects
@@
 		(on_board yes)
 		(dnp no)
-		(property "Reference" "#PWR01206"
+		(property "Reference" "#PWR1206"
 			(at 128.27 116.84 0)
 			(effects
@@
 			(project "sax2"
 				(path "/6c8448b4-b04d-47e1-934e-e40cbe27a7be/095cddf1-6522-4d3b-885d-b21acd91d0c6"
-					(reference "#PWR01206")
-					(unit 1)
-				)
-			)
-		)
-	)
-	(symbol
-		(lib_id "V2_Device:R_0603_10k")
+					(reference "#PWR1206")
+					(unit 1)
+				)
+			)
+		)
+	)
+	(symbol
+		(lib_id "V2_Resistor:0603_10k")
 		(at 172.72 102.87 0)
 		(unit 1)
@@
 		(on_board yes)
 		(dnp no)
-		(property "Reference" "#PWR01207"
+		(property "Reference" "#PWR1207"
 			(at 148.59 121.92 0)
 			(effects
@@
 			(project "sax2"
 				(path "/6c8448b4-b04d-47e1-934e-e40cbe27a7be/095cddf1-6522-4d3b-885d-b21acd91d0c6"
-					(reference "#PWR01207")
-					(unit 1)
-				)
-			)
-		)
-	)
-	(symbol
-		(lib_id "V2_Device:C_1210_10u")
+					(reference "#PWR1207")
+					(unit 1)
+				)
+			)
+		)
+	)
+	(symbol
+		(lib_id "V2_Capacitor:1210_10u")
 		(at 97.79 97.79 0)
 		(unit 1)

Commit message: Update
Parts:
- C1203, C1204: value 10u -> 22u
Changed lines of the file:
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@@
 			)
 		)
-		(property "Value" "10u"
+		(property "Value" "22u"
 			(at 198.12 99.06 0)
 			(effects
@@
 			)
 		)
-		(property "Value" "10u"
+		(property "Value" "22u"
 			(at 187.96 98.806 0)
 			(effects
