File: hardware/sax2/sax2.kicad_pcb (KiCad board)
At the start: 4 copper layers, 80 x 34.5 mm, 105 parts, among them IC1401 MP3V5004GP, J101 Cortex_Debug, J102 DX07S016JA3, J1101 NE8FAH, J1301 2x05_Horizontal, SW101 SKSG, SW102 SKSG, U101 TPS78433QWDRBRQ1, U102 ATSAMD51J, U1101 THVD2442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

Commit message: Refresh
Changed lines of the file:
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@@
 		)
 		(fp_line
-			(start -3.175 -1.2)
-			(end -3.175 -3.7)
-			(stroke
-				(width 0.127)
-				(type solid)
-			)
-			(layer "F.SilkS")
-		)
-		(fp_line
 			(start 3.175 -1.2)
 			(end -3.175 -1.2)
 			(stroke
-				(width 0.127)
+				(width 0.1)
 				(type solid)
 			)
@@
 			(end -2.54 -3.7)
 			(stroke
-				(width 0.127)
+				(width 0.1)
 				(type solid)
 			)
@@
 			(end -1.27 -3.7)
 			(stroke
-				(width 0.127)
+				(width 0.1)
 				(type solid)
 			)
@@
 			(end 2.54 -3.7)
 			(stroke
-				(width 0.127)
+				(width 0.1)
 				(type solid)
 			)
@@
 			(end 3.175 -3.7)
 			(stroke
-				(width 0.127)
-				(type solid)
-			)
-			(layer "F.SilkS")
-		)
-		(fp_line
-			(start 3.175 -3.7)
-			(end 3.175 -1.2)
-			(stroke
-				(width 0.127)
+				(width 0.1)
 				(type solid)
 			)
@@
 			(effects
 				(font
-					(size 0.75 0.75)
+					(size 0.5 0.5)
 					(thickness 0.1)
 					(bold yes)
@@
 		)
 		(embedded_fonts no)
-		(model "../../3dmodels/V2_Connector_PinHeader_1.27mm.3dshapes/PinHeader_2x05_P1.27mm.stp"
+		(model "../../3dmodels/V2_Connector_PinHeader_1.27mm.3dshapes/PinHeader_2x05_P1.27mm_Horizontal.step"
 			(offset
 				(xyz 2.52 1.18 1.65)
@@
 			(effects
 				(font
-					(size 0.75 0.75)
+					(size 0.5 0.5)
 					(thickness 0.1)
 				)
@@
 			(effects
 				(font
-					(size 0.75 0.75)
+					(size 0.5 0.5)
 					(thickness 0.1)
 				)
@@
 				(font
 					(size 0.5 0.5)
-					(thickness 0.05)
+					(thickness 0.1)
+					(bold yes)
 				)
 			)
@@
 				(font
 					(size 0.5 0.5)
-					(thickness 0.05)
+					(thickness 0.1)
+					(bold yes)
 				)
 			)
@@
 		)
 		(pad "" smd roundrect
-			(at -0.876812 1.006939)
-			(size 0.513878 0.846374)
+			(at -0.875 0.25)
+			(size 0.48 0.85)
 			(layers "F.Paste")
-			(roundrect_rratio 0.1)
+			(roundrect_rratio 0.15)
 		)
 		(pad "" smd roundrect
-			(at -0.875 0.25)
-			(size 0.5 0.85)
+			(at -0.875 1)
+			(size 0.48 0.85)
 			(layers "F.Paste")
-			(roundrect_rratio 0.1)
+			(roundrect_rratio 0.15)
 		)
 		(pad "" smd roundrect
 			(at -0.875 1.75)
-			(size 0.5 0.85)
+			(size 0.48 0.85)
 			(layers "F.Paste")
-			(roundrect_rratio 0.1)
+			(roundrect_rratio 0.15)
 		)
 		(pad "" smd roundrect
@@
 		(pad "" smd roundrect
 			(at 0.875 0.25)
-			(size 0.5 0.85)
+			(size 0.48 0.85)
 			(layers "F.Paste")
-			(roundrect_rratio 0.1)
+			(roundrect_rratio 0.15)
 		)
 		(pad "" smd roundrect
-			(at 0.876435 1.012691)
-			(size 0.512076 0.847129)
+			(at 0.875 1)
+			(size 0.48 0.85)
 			(layers "F.Paste")
-			(roundrect_rratio 0.1)
+			(roundrect_rratio 0.15)
 		)
 		(pad "" smd roundrect
-			(at 0.877396 1.75)
-			(size 0.5 0.845206)
+			(at 0.875 1.75)
+			(size 0.48 0.85)
 			(layers "F.Paste")
-			(roundrect_rratio 0.1)
+			(roundrect_rratio 0.15)
 		)
 		(pad "" smd roundrect
@@
 		)
 		(pad "1" smd roundrect
-			(at -0.7875 0 90)
-			(size 0.875 0.95)
+			(at -0.825 0 90)
+			(size 0.8 0.8)
 			(layers "F.Cu" "F.Mask" "F.Paste")
-			(roundrect_rratio 0.25)
+			(roundrect_rratio 0.125)
 			(net 12 "Net-(D102-K)")
 			(pinfunction "K")
@@
 		)
 		(pad "2" smd roundrect
-			(at 0.7875 0 90)
-			(size 0.875 0.95)
+			(at 0.825 0 90)
+			(size 0.8 0.8)
 			(layers "F.Cu" "F.Mask" "F.Paste")
-			(roundrect_rratio 0.25)
+			(roundrect_rratio 0.125)
 			(net 14 "/LED-Onboard")
 			(pinfunction "A")
@@
 			(effects
 				(font
-					(size 0.75 0.75)
+					(size 0.5 0.5)
 					(thickness 0.1)
 				)
@@
 	)
 	(gr_line
-		(start 138.75 108.25)
-		(end 142 108.25)
+		(start 62.5 84)
+		(end 62.5 116.5)
+		(stroke
+			(width 0.05)
+			(type solid)
+		)
+		(layer "Edge.Cuts")
+	)
+	(gr_arc
+		(start 62.5 84)
+		(mid 62.792893 83.292893)
+		(end 63.5 83)
 		(stroke
 			(width 0.05)
@@
 	)
 	(gr_line
-		(start 138.75 108.25)
-		(end 138.75 106.25)
+		(start 63.5 83)
+		(end 141.5 83)
 		(stroke
 			(width 0.05)
@@
 	)
 	(gr_arc
-		(start 142.5 105.75)
-		(mid 142.353553 106.103553)
-		(end 142 106.25)
+		(start 63.5 117.5)
+		(mid 62.792893 117.207107)
+		(end 62.5 116.5)
 		(stroke
 			(width 0.05)
@@
 	)
 	(gr_line
-		(start 62.5 84)
-		(end 62.5 116.5)
+		(start 63.5 117.5)
+		(end 141.5 117.5)
 		(stroke
 			(width 0.05)
@@
 	)
 	(gr_line
-		(start 63.5 83)
-		(end 141.5 83)
+		(start 138.75 106.25)
+		(end 142 106.25)
 		(stroke
 			(width 0.05)
@@
 		(layer "Edge.Cuts")
 	)
-	(gr_arc
-		(start 142 108.25)
-		(mid 142.353553 108.396447)
-		(end 142.5 108.75)
+	(gr_line
+		(start 138.75 108.25)
+		(end 138.75 106.25)
 		(stroke
 			(width 0.05)
@@
 	)
 	(gr_line
-		(start 142.5 84)
-		(end 142.5 105.75)
+		(start 138.75 108.25)
+		(end 142 108.25)
 		(stroke
 			(width 0.05)
@@
 	)
 	(gr_arc
-		(start 63.5 117.5)
-		(mid 62.792893 117.207107)
-		(end 62.5 116.5)
+		(start 141.5 83)
+		(mid 142.207107 83.292893)
+		(end 142.5 84)
 		(stroke
 			(width 0.05)
@@
 	)
 	(gr_arc
-		(start 142.5 116.5)
-		(mid 142.207107 117.207107)
-		(end 141.5 117.5)
+		(start 142 108.25)
+		(mid 142.353553 108.396447)
+		(end 142.5 108.75)
 		(stroke
 			(width 0.05)
@@
 	)
 	(gr_line
-		(start 138.75 106.25)
-		(end 142 106.25)
+		(start 142.5 84)
+		(end 142.5 105.75)
 		(stroke
 			(width 0.05)
@@
 	)
 	(gr_arc
-		(start 62.5 84)
-		(mid 62.792893 83.292893)
-		(end 63.5 83)
+		(start 142.5 105.75)
+		(mid 142.353553 106.103553)
+		(end 142 106.25)
 		(stroke
 			(width 0.05)
@@
 	)
 	(gr_arc
-		(start 141.5 83)
-		(mid 142.207107 83.292893)
-		(end 142.5 84)
-		(stroke
-			(width 0.05)
-			(type solid)
-		)
-		(layer "Edge.Cuts")
-	)
-	(gr_line
-		(start 63.5 117.5)
+		(start 142.5 116.5)
+		(mid 142.207107 117.207107)
 		(end 141.5 117.5)
 		(stroke

Commit message: Update library
Parts:
- TVS101: value SMBJ36CA -> SMBJ33CA
Connections:
- net +24V renamed /+VLINK-Supply
- net /+24V-Link renamed +VLINK

Commit message: Update library
Parts:
- J101: value Cortex_Debug -> Cortex; footprint V2_Cortex_Debug:Cortex_Debug_Pad -> V2_Connector_Debug:Cortex
- U1201: value TPSM33625 -> TPSM365R6FRDNR; footprint V2_Converter_DCDC:TPSM33625 -> V2_Converter_DCDC:QFN-11
Routing:
- net /SWCLK: track 7.86 -> 16.4 mm, vias 2 -> 0
- net GND: vias 124 -> 122
- net +3V3: vias 23 -> 22
