File: hardware/sax2/sax2.kicad_pcb (KiCad board)
At the start: 4 copper layers, 80 x 34.5 mm, 105 parts, among them IC1401 MP3V5004GP, J101 Cortex, J102 DX07S016JA3, J1101 NE8FAH, J1301 2x05_Horizontal, SW101 SKSG, SW102 SKSG, U101 TPS78433QWDRBRQ1, U102 ATSAMD51J, U1101 THVD2442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

Commit message: Update Library
Parts:
- C1203, C1204: value 22u -> 10u

Commit message: Update
Parts:
- C1203, C1204: value 10u -> 22u

Commit message: Update
Connections:
- net /SCK renamed /SCL
