File: hardware/sax2/sax2.kicad_sch (KiCad schematic)
At the start: 36 parts, among them J101 Cortex_Debug, J102 DX07S016JA3, SW101 SKSG, SW102 SKSG, U101 TPS78433QWDRBRQ1, U102 ATSAMD51J, Y101 32k768

Commit message: Refresh footprints
Parts:
- D102: Mouser 755-SML-D12M8WT86C -> 755-SML-D12D1WT86; Product SML-D12M8WT86C -> SML-D12D1WT86
Changed lines of the file:
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@@
 		(at 233.68 152.4 0)
 		(unit 1)
-		(exclude_from_sim yes)
+		(exclude_from_sim no)
 		(in_bom no)
 		(on_board yes)
@@
 			)
 		)
-		(property "Mouser" "755-SML-D12M8WT86C"
+		(property "Mouser" "755-SML-D12D1WT86"
 			(at 132.08 66.04 0)
 			(effects
@@
 			)
 		)
-		(property "Product" "SML-D12M8WT86C "
+		(property "Product" "SML-D12D1WT86"
 			(at 132.08 71.12 0)
 			(effects
@@
 		(at 123.19 99.06 0)
 		(unit 1)
-		(exclude_from_sim yes)
+		(exclude_from_sim no)
 		(in_bom no)
 		(on_board yes)
@@
 			)
 		)
-		(property "Description" "Power symbol creates a global label with name \"Earth\""
+		(property "Description" "Power symbol creates a global label with name \"Shield\""
 			(at 250.19 83.82 0)
 			(effects
@@
 			)
 		)
-		(property "Description" "Power symbol creates a global label with name \"Earth\""
+		(property "Description" "Power symbol creates a global label with name \"Shield\""
 			(at 172.72 119.38 0)
 			(effects
@@
 		(at 208.28 153.67 0)
 		(unit 1)
-		(exclude_from_sim yes)
+		(exclude_from_sim no)
 		(in_bom no)
 		(on_board yes)

Commit message: Update library
Parts:
- C101: Rating (none) -> 10V
- C102, C103, C104, C105, C106, C111: Rating (none) -> 50V
- TVS101: value SMBJ36CA -> SMBJ33CA; symbol V2_Diode:SMBJ36CA -> V2_Diode:SMBJ33CA; Mouser 652-SMBJ36CA-Q -> 652-SMBJ33CA-Q; Product SMBJ36CA-Q -> SMBJ33CA-Q; Rating 36V -> 33V
Connections:
- net +24V renamed +VLINK-Supply
- net +24V-Link renamed +VLINK
Other:
- moved on the sheet: C111, D104, D105, TVS101

Commit message: Update library
Parts:
- J101: value Cortex_Debug -> Cortex; footprint V2_Cortex_Debug:Cortex_Debug_Pad -> V2_Connector_Debug:Cortex; symbol V2_Cortex_Debug:Cortex_Debug -> V2_Connector_Debug:Cortex
Changed lines of the file:
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@@
 		(at 233.68 152.4 0)
 		(unit 1)
-		(exclude_from_sim no)
+		(exclude_from_sim yes)
 		(in_bom no)
 		(on_board yes)
@@
 			)
 		)
-		(property "Sim.Enable" "0"
-			(at 233.68 152.4 0)
-			(effects
-				(font
-					(size 1.27 1.27)
-				)
-				(hide yes)
-			)
-		)
 		(instances
 			(project ""
@@
 	)
 	(symbol
-		(lib_id "V2_Cortex_Debug:Cortex_Debug")
+		(lib_id "V2_Connector_Debug:Cortex")
 		(at 123.19 99.06 0)
 		(unit 1)
@@
 			)
 		)
-		(property "Value" "Cortex_Debug"
+		(property "Value" "Cortex"
 			(at 124.46 88.9 0)
 			(effects
@@
 			)
 		)
-		(property "Footprint" "V2_Cortex_Debug:Cortex_Debug_Pad"
+		(property "Footprint" "V2_Connector_Debug:Cortex"
 			(at 123.19 113.03 0)
 			(effects
@@
 		(at 208.28 153.67 0)
 		(unit 1)
-		(exclude_from_sim no)
+		(exclude_from_sim yes)
 		(in_bom no)
 		(on_board yes)
@@
 			(at 208.28 153.67 0)
 			(effects
-				(font
-					(size 1.27 1.27)
-				)
-				(hide yes)
-			)
-		)
-		(property "Sim.Enable" "0"
-			(at 208.28 153.67 0)
-			(effects
