File: hardware/sax2/sax2.kicad_sch (KiCad schematic)
At the start: 36 parts, among them J101 Cortex, J102 DX07S016JA3, SW101 SKSG, SW102 SKSG, U101 TPS78433QWDRBRQ1, U102 ATSAMD51J, Y101 32k768

Commit message: Replace Order_Number
Parts:
- H101: value MountingHole_2mm -> 2mm
- INFO101: value Order_Number -> (none); footprint V2_Production:Order_Number -> V2_Production:Revision; symbol V2_Production:Order_Number -> V2_Production:Revision
Changed lines of the file:
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@@
 		(at 233.68 152.4 0)
 		(unit 1)
-		(exclude_from_sim yes)
+		(exclude_from_sim no)
 		(in_bom no)
 		(on_board yes)
@@
 			)
 		)
-		(property "Value" "MountingHole_2mm"
+		(property "Value" "2mm"
 			(at 236.22 153.6699 0)
 			(effects
@@
 	)
 	(symbol
-		(lib_id "V2_Production:Order_Number")
+		(lib_id "V2_Production:Revision")
 		(at 213.36 168.91 0)
 		(unit 1)
@@
 			)
 		)
-		(property "Value" "Order_Number"
+		(property "Value" ""
 			(at 213.36 171.45 0)
 			(effects
@@
 			)
 		)
-		(property "Footprint" "V2_Production:Order_Number"
+		(property "Footprint" "V2_Production:Revision"
 			(at 213.36 173.99 0)
 			(effects
@@
 		(at 208.28 153.67 0)
 		(unit 1)
-		(exclude_from_sim yes)
+		(exclude_from_sim no)
 		(in_bom no)
 		(on_board yes)

Commit message: Update Library
Parts:
- C101: symbol V2_Device:C_0603_10u -> V2_Capacitor:0603_10u
- C102, C103, C104, C105, C106, C111: symbol V2_Device:C_0603_0u1 -> V2_Capacitor:0603_0u1
- C107, C110: symbol V2_Device:C_0603_18p -> V2_Capacitor:0603_18p
- C108, C109: symbol V2_Device:C_0805_10u -> V2_Capacitor:0805_10u
- D102: symbol V2_Device:LED_0603_Orange -> V2_LED:0603_Orange
- INFO101: value (none) -> ~
- R101: symbol V2_Device:R_0603_330R -> V2_Resistor:0603_330R
- R102, R103: symbol V2_Device:R_0603_5k1 -> V2_Resistor:0603_5k1
- R104: symbol V2_Device:R_0603_100k -> V2_Resistor:0603_100k
- Y101: symbol V2_Device:Crystal_3.2x1.5_32k768 -> V2_Crystal:3.2x1.5_32k768

Commit message: Update
Parts:
- INFO101: value ~ -> (none)
Changed lines of the file:
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@@
 			)
 		)
-		(property "Value" "~"
+		(property "Value" ""
 			(at 213.36 171.45 0)
 			(effects

Commit message: Update
Parts:
- INFO101: value (none) -> ~
Connections:
- net SCK renamed SCL
Changed lines of the file:
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@@
 	(title_block
 		(title "V2 sax")
-		(date "2026-02-10")
+		(date "2026-02-18")
 		(rev "2026-02-10")
 		(company "Versio Duo")
@@
 	(wire
 		(pts
-			(xy 251.46 50.8) (xy 270.51 50.8)
+			(xy 251.46 50.8) (xy 271.78 50.8)
 		)
 		(stroke
@@
 		)
 	)
-	(label "SCK"
+	(label "SCL"
 		(at 31.75 82.55 0)
 		(effects
@@
 	)
 	(label "LED-Sensor"
-		(at 270.51 50.8 180)
+		(at 271.78 50.8 180)
 		(effects
 			(font
@@
 		)
 	)
-	(label "SCK"
+	(label "SCL"
 		(at 134.62 152.4 180)
 		(effects
@@
 		)
 		(property "Value" "+3V3"
-			(at 194.31 35.56 0)
+			(at 198.12 34.798 0)
 			(effects
 				(font
 					(size 1.27 1.27)
+					(color 255 92 187 1)
 				)
-				(justify left)
 			)
 		)
@@
 		)
 		(property "Value" "+5V"
-			(at 268.478 121.92 90)
+			(at 268.986 121.92 90)
 			(effects
 				(font
 					(size 1.27 1.27)
+					(color 255 92 187 1)
 				)
 			)
@@
 		)
 		(property "Value" "+5V"
-			(at 258.572 48.26 90)
+			(at 257.302 48.26 90)
 			(effects
 				(font
 					(size 1.27 1.27)
+					(color 255 92 187 1)
 				)
-				(justify right)
 			)
 		)
@@
 		(on_board yes)
 		(dnp no)
-		(fields_autoplaced yes)
 		(property "Reference" "#PWR120"
 			(at 246.38 83.82 0)
@@
 		)
 		(property "Value" "+5V"
-			(at 254 83.8199 90)
+			(at 255.778 83.8199 90)
 			(effects
 				(font
 					(size 1.27 1.27)
+					(color 255 92 187 1)
 				)
-				(justify left)
 			)
 		)
@@
 		)
 		(property "Value" "+3V3"
-			(at 49.53 45.72 90)
+			(at 49.53 45.72 0)
 			(effects
 				(font
 					(size 1.27 1.27)
+					(color 255 92 187 1)
 				)
-				(justify left bottom)
 			)
 		)
@@
 		)
 		(property "Value" "+5V"
-			(at 173.99 35.56 0)
+			(at 173.99 34.798 0)
 			(effects
 				(font
 					(size 1.27 1.27)
+					(color 255 92 187 1)
 				)
 			)
@@
 			)
 		)
-		(property "Value" ""
+		(property "Value" "~"
 			(at 213.36 171.45 0)
 			(effects
@@
 		(on_board yes)
 		(dnp no)
-		(fields_autoplaced yes)
 		(property "Reference" "#PWR123"
 			(at 115.57 93.98 0)
@@
 		)
 		(property "Value" "+3V3"
-			(at 107.95 93.9799 90)
+			(at 104.648 93.9799 90)
 			(effects
 				(font
 					(size 1.27 1.27)
+					(color 255 92 187 1)
 				)
-				(justify left)
 			)
 		)
@@
 		(on_board yes)
 		(dnp no)
-		(fields_autoplaced yes)
 		(property "Reference" "#PWR119"
 			(at 205.74 83.82 0)
@@
 		)
 		(property "Value" "+5V"
-			(at 213.36 83.8199 90)
+			(at 214.884 83.8199 90)
 			(effects
 				(font
 					(size 1.27 1.27)
+					(color 255 92 187 1)
 				)
-				(justify left)
 			)
 		)
@@
 				(font
 					(size 1.27 1.27)
+					(color 255 92 187 1)
 				)
 			)
@@
 		)
 		(property "Value" "+3V3"
-			(at 44.45 120.65 90)
+			(at 41.656 120.65 90)
 			(effects
 				(font
 					(size 1.27 1.27)
+					(color 255 92 187 1)
 				)
-				(justify left)
 			)
 		)
