File: hardware/sax2/ExpressionInput.kicad_sch (KiCad schematic)
At the start: 5 parts

Commit message: Update Library
Parts:
- C1405: symbol V2_Device:C_0603_0u022 -> V2_Capacitor:0603_0u022
- R1403: symbol V2_Device:R_0603_1k -> V2_Resistor:0603_1k
- R1405: symbol V2_Device:R_0603_100k -> V2_Resistor:0603_100k
Changed lines of the file:
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@@
 	)
 	(symbol
-		(lib_id "V2_Device:R_0603_1k")
+		(lib_id "V2_Resistor:0603_1k")
 		(at 137.16 92.71 270)
 		(unit 1)
@@
 		(dnp no)
 		(fields_autoplaced yes)
-		(property "Reference" "#PWR01414"
+		(property "Reference" "#PWR1414"
 			(at 123.19 104.14 0)
 			(effects
@@
 			(project "sax2"
 				(path "/6c8448b4-b04d-47e1-934e-e40cbe27a7be/986c2710-b6fb-48af-9291-0e7dc7b5abf9/09fde53a-0726-4a1a-ba32-997a9c8cb2ac"
-					(reference "#PWR01701")
+					(reference "#PWR1701")
 					(unit 1)
 				)
 				(path "/6c8448b4-b04d-47e1-934e-e40cbe27a7be/986c2710-b6fb-48af-9291-0e7dc7b5abf9/75bdefb6-cbec-430c-b2f6-bba8982a1e16"
-					(reference "#PWR01414")
+					(reference "#PWR1414")
 					(unit 1)
 				)
 				(path "/6c8448b4-b04d-47e1-934e-e40cbe27a7be/986c2710-b6fb-48af-9291-0e7dc7b5abf9/7eddc4ac-e264-4e8d-993d-81fc85f367c8"
-					(reference "#PWR01501")
+					(reference "#PWR1501")
 					(unit 1)
 				)
 				(path "/6c8448b4-b04d-47e1-934e-e40cbe27a7be/986c2710-b6fb-48af-9291-0e7dc7b5abf9/ab1436ac-5052-4cae-b140-374128cd8279"
-					(reference "#PWR02101")
+					(reference "#PWR2101")
 					(unit 1)
 				)
 				(path "/6c8448b4-b04d-47e1-934e-e40cbe27a7be/986c2710-b6fb-48af-9291-0e7dc7b5abf9/b1b709ba-4565-4658-b8d7-ca720ae6b4d0"
-					(reference "#PWR01901")
+					(reference "#PWR1901")
 					(unit 1)
 				)
 				(path "/6c8448b4-b04d-47e1-934e-e40cbe27a7be/986c2710-b6fb-48af-9291-0e7dc7b5abf9/e5e66090-238e-4b5d-8478-8d0716aa9aa6"
-					(reference "#PWR01601")
+					(reference "#PWR1601")
 					(unit 1)
 				)
 				(path "/6c8448b4-b04d-47e1-934e-e40cbe27a7be/986c2710-b6fb-48af-9291-0e7dc7b5abf9/f153ee55-65c6-4eb1-a6b0-fdf78a9680f1"
-					(reference "#PWR02001")
+					(reference "#PWR2001")
 					(unit 1)
 				)
 				(path "/6c8448b4-b04d-47e1-934e-e40cbe27a7be/986c2710-b6fb-48af-9291-0e7dc7b5abf9/f5d1679c-7076-43d7-b0e0-c560820060c0"
-					(reference "#PWR01801")
+					(reference "#PWR1801")
 					(unit 1)
 				)
@@
 		(dnp no)
 		(fields_autoplaced yes)
-		(property "Reference" "#PWR01423"
+		(property "Reference" "#PWR1423"
 			(at 156.21 125.73 0)
 			(effects
@@
 			(project "sax2"
 				(path "/6c8448b4-b04d-47e1-934e-e40cbe27a7be/986c2710-b6fb-48af-9291-0e7dc7b5abf9/09fde53a-0726-4a1a-ba32-997a9c8cb2ac"
-					(reference "#PWR01704")
+					(reference "#PWR1704")
 					(unit 1)
 				)
 				(path "/6c8448b4-b04d-47e1-934e-e40cbe27a7be/986c2710-b6fb-48af-9291-0e7dc7b5abf9/75bdefb6-cbec-430c-b2f6-bba8982a1e16"
-					(reference "#PWR01423")
+					(reference "#PWR1423")
 					(unit 1)
 				)
 				(path "/6c8448b4-b04d-47e1-934e-e40cbe27a7be/986c2710-b6fb-48af-9291-0e7dc7b5abf9/7eddc4ac-e264-4e8d-993d-81fc85f367c8"
-					(reference "#PWR01504")
+					(reference "#PWR1504")
 					(unit 1)
 				)
 				(path "/6c8448b4-b04d-47e1-934e-e40cbe27a7be/986c2710-b6fb-48af-9291-0e7dc7b5abf9/ab1436ac-5052-4cae-b140-374128cd8279"
-					(reference "#PWR02104")
+					(reference "#PWR2104")
 					(unit 1)
 				)
 				(path "/6c8448b4-b04d-47e1-934e-e40cbe27a7be/986c2710-b6fb-48af-9291-0e7dc7b5abf9/b1b709ba-4565-4658-b8d7-ca720ae6b4d0"
-					(reference "#PWR01904")
+					(reference "#PWR1904")
 					(unit 1)
 				)
 				(path "/6c8448b4-b04d-47e1-934e-e40cbe27a7be/986c2710-b6fb-48af-9291-0e7dc7b5abf9/e5e66090-238e-4b5d-8478-8d0716aa9aa6"
-					(reference "#PWR01604")
+					(reference "#PWR1604")
 					(unit 1)
 				)
 				(path "/6c8448b4-b04d-47e1-934e-e40cbe27a7be/986c2710-b6fb-48af-9291-0e7dc7b5abf9/f153ee55-65c6-4eb1-a6b0-fdf78a9680f1"
-					(reference "#PWR02004")
+					(reference "#PWR2004")
 					(unit 1)
 				)
 				(path "/6c8448b4-b04d-47e1-934e-e40cbe27a7be/986c2710-b6fb-48af-9291-0e7dc7b5abf9/f5d1679c-7076-43d7-b0e0-c560820060c0"
-					(reference "#PWR01804")
+					(reference "#PWR1804")
 					(unit 1)
 				)
@@
 		(dnp no)
 		(fields_autoplaced yes)
-		(property "Reference" "#PWR01416"
+		(property "Reference" "#PWR1416"
 			(at 180.34 104.14 0)
 			(effects
@@
 			(project "sax2"
 				(path "/6c8448b4-b04d-47e1-934e-e40cbe27a7be/986c2710-b6fb-48af-9291-0e7dc7b5abf9/09fde53a-0726-4a1a-ba32-997a9c8cb2ac"
-					(reference "#PWR01702")
+					(reference "#PWR1702")
 					(unit 1)
 				)
 				(path "/6c8448b4-b04d-47e1-934e-e40cbe27a7be/986c2710-b6fb-48af-9291-0e7dc7b5abf9/75bdefb6-cbec-430c-b2f6-bba8982a1e16"
-					(reference "#PWR01416")
+					(reference "#PWR1416")
 					(unit 1)
 				)
 				(path "/6c8448b4-b04d-47e1-934e-e40cbe27a7be/986c2710-b6fb-48af-9291-0e7dc7b5abf9/7eddc4ac-e264-4e8d-993d-81fc85f367c8"
-					(reference "#PWR01502")
+					(reference "#PWR1502")
 					(unit 1)
 				)
 				(path "/6c8448b4-b04d-47e1-934e-e40cbe27a7be/986c2710-b6fb-48af-9291-0e7dc7b5abf9/ab1436ac-5052-4cae-b140-374128cd8279"
-					(reference "#PWR02102")
+					(reference "#PWR2102")
 					(unit 1)
 				)
 				(path "/6c8448b4-b04d-47e1-934e-e40cbe27a7be/986c2710-b6fb-48af-9291-0e7dc7b5abf9/b1b709ba-4565-4658-b8d7-ca720ae6b4d0"
-					(reference "#PWR01902")
+					(reference "#PWR1902")
 					(unit 1)
 				)
 				(path "/6c8448b4-b04d-47e1-934e-e40cbe27a7be/986c2710-b6fb-48af-9291-0e7dc7b5abf9/e5e66090-238e-4b5d-8478-8d0716aa9aa6"
-					(reference "#PWR01602")
+					(reference "#PWR1602")
 					(unit 1)
 				)
 				(path "/6c8448b4-b04d-47e1-934e-e40cbe27a7be/986c2710-b6fb-48af-9291-0e7dc7b5abf9/f153ee55-65c6-4eb1-a6b0-fdf78a9680f1"
-					(reference "#PWR02002")
+					(reference "#PWR2002")
 					(unit 1)
 				)
 				(path "/6c8448b4-b04d-47e1-934e-e40cbe27a7be/986c2710-b6fb-48af-9291-0e7dc7b5abf9/f5d1679c-7076-43d7-b0e0-c560820060c0"
-					(reference "#PWR01802")
+					(reference "#PWR1802")
 					(unit 1)
 				)
@@
 	)
 	(symbol
-		(lib_id "V2_Device:C_0603_0u022")
+		(lib_id "V2_Capacitor:0603_0u022")
 		(at 180.34 95.25 0)
 		(unit 1)
@@
 		(dnp no)
 		(fields_autoplaced yes)
-		(property "Reference" "#PWR01425"
+		(property "Reference" "#PWR1425"
 			(at 166.37 130.81 0)
 			(effects
@@
 			(project "sax2"
 				(path "/6c8448b4-b04d-47e1-934e-e40cbe27a7be/986c2710-b6fb-48af-9291-0e7dc7b5abf9/09fde53a-0726-4a1a-ba32-997a9c8cb2ac"
-					(reference "#PWR01705")
+					(reference "#PWR1705")
 					(unit 1)
 				)
 				(path "/6c8448b4-b04d-47e1-934e-e40cbe27a7be/986c2710-b6fb-48af-9291-0e7dc7b5abf9/75bdefb6-cbec-430c-b2f6-bba8982a1e16"
-					(reference "#PWR01425")
+					(reference "#PWR1425")
 					(unit 1)
 				)
 				(path "/6c8448b4-b04d-47e1-934e-e40cbe27a7be/986c2710-b6fb-48af-9291-0e7dc7b5abf9/7eddc4ac-e264-4e8d-993d-81fc85f367c8"
-					(reference "#PWR01505")
+					(reference "#PWR1505")
 					(unit 1)
 				)
 				(path "/6c8448b4-b04d-47e1-934e-e40cbe27a7be/986c2710-b6fb-48af-9291-0e7dc7b5abf9/ab1436ac-5052-4cae-b140-374128cd8279"
-					(reference "#PWR02105")
+					(reference "#PWR2105")
 					(unit 1)
 				)
 				(path "/6c8448b4-b04d-47e1-934e-e40cbe27a7be/986c2710-b6fb-48af-9291-0e7dc7b5abf9/b1b709ba-4565-4658-b8d7-ca720ae6b4d0"
-					(reference "#PWR01905")
+					(reference "#PWR1905")
 					(unit 1)
 				)
 				(path "/6c8448b4-b04d-47e1-934e-e40cbe27a7be/986c2710-b6fb-48af-9291-0e7dc7b5abf9/e5e66090-238e-4b5d-8478-8d0716aa9aa6"
-					(reference "#PWR01605")
+					(reference "#PWR1605")
 					(unit 1)
 				)
 				(path "/6c8448b4-b04d-47e1-934e-e40cbe27a7be/986c2710-b6fb-48af-9291-0e7dc7b5abf9/f153ee55-65c6-4eb1-a6b0-fdf78a9680f1"
-					(reference "#PWR02005")
+					(reference "#PWR2005")
 					(unit 1)
 				)
 				(path "/6c8448b4-b04d-47e1-934e-e40cbe27a7be/986c2710-b6fb-48af-9291-0e7dc7b5abf9/f5d1679c-7076-43d7-b0e0-c560820060c0"
-					(reference "#PWR01805")
+					(reference "#PWR1805")
 					(unit 1)
 				)
@@
 		(dnp no)
 		(fields_autoplaced yes)
-		(property "Reference" "#PWR01418"
+		(property "Reference" "#PWR1418"
 			(at 148.59 106.68 0)
 			(effects
@@
 			(project "sax2"
 				(path "/6c8448b4-b04d-47e1-934e-e40cbe27a7be/986c2710-b6fb-48af-9291-0e7dc7b5abf9/09fde53a-0726-4a1a-ba32-997a9c8cb2ac"
-					(reference "#PWR01703")
+					(reference "#PWR1703")
 					(unit 1)
 				)
 				(path "/6c8448b4-b04d-47e1-934e-e40cbe27a7be/986c2710-b6fb-48af-9291-0e7dc7b5abf9/75bdefb6-cbec-430c-b2f6-bba8982a1e16"
-					(reference "#PWR01418")
+					(reference "#PWR1418")
 					(unit 1)
 				)
 				(path "/6c8448b4-b04d-47e1-934e-e40cbe27a7be/986c2710-b6fb-48af-9291-0e7dc7b5abf9/7eddc4ac-e264-4e8d-993d-81fc85f367c8"
-					(reference "#PWR01503")
+					(reference "#PWR1503")
 					(unit 1)
 				)
 				(path "/6c8448b4-b04d-47e1-934e-e40cbe27a7be/986c2710-b6fb-48af-9291-0e7dc7b5abf9/ab1436ac-5052-4cae-b140-374128cd8279"
-					(reference "#PWR02103")
+					(reference "#PWR2103")
 					(unit 1)
 				)
 				(path "/6c8448b4-b04d-47e1-934e-e40cbe27a7be/986c2710-b6fb-48af-9291-0e7dc7b5abf9/b1b709ba-4565-4658-b8d7-ca720ae6b4d0"
-					(reference "#PWR01903")
+					(reference "#PWR1903")
 					(unit 1)
 				)
 				(path "/6c8448b4-b04d-47e1-934e-e40cbe27a7be/986c2710-b6fb-48af-9291-0e7dc7b5abf9/e5e66090-238e-4b5d-8478-8d0716aa9aa6"
-					(reference "#PWR01603")
+					(reference "#PWR1603")
 					(unit 1)
 				)
 				(path "/6c8448b4-b04d-47e1-934e-e40cbe27a7be/986c2710-b6fb-48af-9291-0e7dc7b5abf9/f153ee55-65c6-4eb1-a6b0-fdf78a9680f1"
-					(reference "#PWR02003")
+					(reference "#PWR2003")
 					(unit 1)
 				)
 				(path "/6c8448b4-b04d-47e1-934e-e40cbe27a7be/986c2710-b6fb-48af-9291-0e7dc7b5abf9/f5d1679c-7076-43d7-b0e0-c560820060c0"
-					(reference "#PWR01803")
+					(reference "#PWR1803")
 					(unit 1)
 				)
@@
 	)
 	(symbol
-		(lib_id "V2_Device:R_0603_100k")
+		(lib_id "V2_Resistor:0603_100k")
 		(at 123.19 95.25 0)
 		(unit 1)

Commit message: Update
Changed lines of the file:
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@@
 		(on_board yes)
 		(dnp no)
-		(fields_autoplaced yes)
 		(property "Reference" "#PWR1423"
 			(at 156.21 125.73 0)
@@
 		)
 		(property "Value" "+5V"
-			(at 163.83 126.365 90)
+			(at 166.116 125.603 90)
 			(effects
 				(font
 					(size 1.27 1.27)
+					(color 255 92 187 1)
 				)
-				(justify left)
 			)
 		)
