File: hardware/sax2/LinkPlug.kicad_sch (KiCad schematic)
At the start: 4 parts, among them J1101 NE8FAH, U1101 THVD2442

Commit message: Update library
Parts:
- C1101: Rating (none) -> 50V
Changed lines of the file:
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@@
 			)
 		)
-		(property "Description" "Power symbol creates a global label with name \"GND\" , ground"
+		(property "Description" ""
 			(at 168.91 74.93 0)
 			(effects
@@
 			)
 		)
-		(property "Description" "Power symbol creates a global label with name \"GND\" , ground"
+		(property "Description" ""
 			(at 148.59 107.95 0)
 			(effects
@@
 			)
 		)
-		(property "Description" "Power symbol creates a global label with name \"+3V3\""
+		(property "Description" ""
 			(at 148.59 69.85 0)
 			(effects
@@
 		(property "Product" "CGA3E2X7R1H104M080AA"
 			(at 168.91 90.17 0)
+			(effects
+				(font
+					(size 1.27 1.27)
+				)
+				(hide yes)
+			)
+		)
+		(property "Rating" "50V"
+			(at 168.91 95.25 0)
 			(effects
 				(font
@@
 			)
 		)
-		(property "Description" "Power symbol creates a global label with name \"GND\" , ground"
+		(property "Description" ""
 			(at 138.43 127 0)
 			(effects

Commit message: Update Library
Parts:
- C1101: symbol V2_Device:C_0603_0u1 -> V2_Capacitor:0603_0u1
- R1101: symbol V2_Device:R_0603_100R -> V2_Resistor:0603_100R
Changed lines of the file:
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@@
 		(on_board yes)
 		(dnp no)
-		(property "Reference" "#PWR01102"
+		(property "Reference" "#PWR1102"
 			(at 168.91 81.28 0)
 			(effects
@@
 			(project "sax2"
 				(path "/6c8448b4-b04d-47e1-934e-e40cbe27a7be/be5efeaa-f0dd-4882-b2f8-53c61e0a33bd"
-					(reference "#PWR01102")
+					(reference "#PWR1102")
 					(unit 1)
 				)
@@
 	)
 	(symbol
-		(lib_id "V2_Device:R_0603_100R")
+		(lib_id "V2_Resistor:0603_100R")
 		(at 161.29 87.63 0)
 		(unit 1)
@@
 		(on_board yes)
 		(dnp no)
-		(property "Reference" "#PWR01103"
+		(property "Reference" "#PWR1103"
 			(at 148.59 114.3 0)
 			(effects
@@
 			(project "sax2"
 				(path "/6c8448b4-b04d-47e1-934e-e40cbe27a7be/be5efeaa-f0dd-4882-b2f8-53c61e0a33bd"
-					(reference "#PWR01103")
+					(reference "#PWR1103")
 					(unit 1)
 				)
@@
 		(on_board yes)
 		(dnp no)
-		(property "Reference" "#PWR01101"
+		(property "Reference" "#PWR1101"
 			(at 148.59 73.66 0)
 			(effects
@@
 			(project "sax2"
 				(path "/6c8448b4-b04d-47e1-934e-e40cbe27a7be/be5efeaa-f0dd-4882-b2f8-53c61e0a33bd"
-					(reference "#PWR01101")
+					(reference "#PWR1101")
 					(unit 1)
 				)
@@
 	)
 	(symbol
-		(lib_id "V2_Device:C_0603_0u1")
+		(lib_id "V2_Capacitor:0603_0u1")
 		(at 168.91 72.39 0)
 		(unit 1)
@@
 		(on_board yes)
 		(dnp no)
-		(property "Reference" "#PWR01104"
+		(property "Reference" "#PWR1104"
 			(at 132.08 127 0)
 			(effects
@@
 			(project "sax2"
 				(path "/6c8448b4-b04d-47e1-934e-e40cbe27a7be/be5efeaa-f0dd-4882-b2f8-53c61e0a33bd"
-					(reference "#PWR01104")
-					(unit 1)
-				)
+					(reference "#PWR1104")
+					(unit 1)
+				)
