File: hardware/sax2/OrientationSensor.kicad_sch (KiCad schematic)
At the start: 10 parts, among them U1401 BMM150, U1402 BHI160

Commit message: Update library
Parts:
- C1401: Rating (none) -> 10V
- C1404: Rating (none) -> 50V
Changed lines of the file:
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@@
+			)
+		)
+		(property "Rating" "10V"
+			(at 129.54 105.41 0)
+			(effects
+				(font
+					(size 1.27 1.27)
+				)
+				(hide yes)
 			)
 		)
@@
 			)
 		)
-		(property "Description" "Power symbol creates a global label with name \"+3V3\""
+		(property "Description" ""
 			(at 93.98 83.82 0)
 			(effects
@@
 			)
 		)
-		(property "Description" "Power symbol creates a global label with name \"+3V3\""
+		(property "Description" ""
 			(at 124.46 77.47 0)
 			(effects
@@
 			)
 		)
-		(property "Description" "Power symbol creates a global label with name \"GND\" , ground"
+		(property "Description" ""
 			(at 160.02 146.05 0)
 			(effects
@@
 			)
 		)
-		(property "Description" "Power symbol creates a global label with name \"GND\" , ground"
+		(property "Description" ""
 			(at 132.08 97.79 0)
 			(effects
@@
 			)
 		)
-		(property "Description" "Power symbol creates a global label with name \"GND\" , ground"
+		(property "Description" ""
 			(at 208.28 106.68 0)
 			(effects
@@
 			)
 		)
+		(property "Rating" "50V"
+			(at 213.36 116.84 0)
+			(effects
+				(font
+					(size 1.27 1.27)
+				)
+				(hide yes)
+			)
+		)
 		(pin "1"
 		)
@@
 			)
 		)
-		(property "Description" "Power symbol creates a global label with name \"GND\" , ground"
+		(property "Description" ""
 			(at 213.36 95.25 0)
 			(effects
@@
 			)
 		)
-		(property "Description" "Power symbol creates a global label with name \"GND\" , ground"
+		(property "Description" ""
 			(at 129.54 82.55 0)
 			(effects
@@
 			)
 		)
-		(property "Description" "Power symbol creates a global label with name \"+3V3\""
+		(property "Description" ""
 			(at 149.86 93.98 0)
 			(effects
@@
 			)
 		)
-		(property "Description" "Power symbol creates a global label with name \"+3V3\""
+		(property "Description" ""
 			(at 190.5 106.68 0)
 			(effects
@@
 			)
 		)
-		(property "Description" "Power symbol creates a global label with name \"GND\" , ground"
+		(property "Description" ""
 			(at 190.5 99.06 0)
 			(effects
@@
 			)
 		)
-		(property "Description" "Power symbol creates a global label with name \"GND\" , ground"
+		(property "Description" ""
 			(at 190.5 93.98 0)
 			(effects
@@
 			)
 		)
-		(property "Description" "Power symbol creates a global label with name \"+3V3\""
+		(property "Description" ""
 			(at 213.36 91.44 0)
 			(effects
@@
 			)
 		)
-		(property "Description" "Power symbol creates a global label with name \"GND\" , ground"
+		(property "Description" ""
 			(at 104.14 107.95 0)
 			(effects
@@
 			)
 		)
-		(property "Description" "Power symbol creates a global label with name \"+5V\""
+		(property "Description" ""
 			(at 160.02 140.97 0)
 			(effects
@@
 			)
 		)
-		(property "Description" "Power symbol creates a global label with name \"GND\" , ground"
+		(property "Description" ""
 			(at 124.46 113.03 0)
 			(effects

Commit message: Update Library
Parts:
- C1401: symbol V2_Device:C_0603_10u -> V2_Capacitor:0603_10u
- C1404: symbol V2_Device:C_0603_0u1 -> V2_Capacitor:0603_0u1
- C1406: symbol V2_Device:C_0603_0u47 -> V2_Capacitor:0603_0u47
- R1401, R1402, R1406, R1407: symbol V2_Device:R_0603_2k7 -> V2_Resistor:0603_2k7
Changed lines of the file:
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@@
 	)
 	(symbol
-		(lib_id "V2_Device:C_0603_10u")
+		(lib_id "V2_Capacitor:0603_10u")
 		(at 129.54 80.01 0)
 		(unit 1)
@@
 	)
 	(symbol
-		(lib_id "V2_Device:R_0603_2k7")
+		(lib_id "V2_Resistor:0603_2k7")
 		(at 95.25 86.36 0)
 		(unit 1)
@@
 		(on_board yes)
 		(dnp no)
-		(property "Reference" "#PWR01403"
+		(property "Reference" "#PWR1403"
 			(at 93.98 87.63 0)
 			(effects
@@
 			(project "sax2"
 				(path "/6c8448b4-b04d-47e1-934e-e40cbe27a7be/f7096e67-1c66-4074-b306-32741be5ff9b"
-					(reference "#PWR01403")
-					(unit 1)
-				)
-			)
-		)
-	)
-	(symbol
-		(lib_id "V2_Device:R_0603_2k7")
+					(reference "#PWR1403")
+					(unit 1)
+				)
+			)
+		)
+	)
+	(symbol
+		(lib_id "V2_Resistor:0603_2k7")
 		(at 148.59 96.52 0)
 		(unit 1)
@@
 	)
 	(symbol
-		(lib_id "V2_Device:R_0603_2k7")
+		(lib_id "V2_Resistor:0603_2k7")
 		(at 92.71 86.36 0)
 		(unit 1)
@@
 		(on_board yes)
 		(dnp no)
-		(property "Reference" "#PWR01401"
+		(property "Reference" "#PWR1401"
 			(at 124.46 81.28 0)
 			(effects
@@
 			(project "sax2"
 				(path "/6c8448b4-b04d-47e1-934e-e40cbe27a7be/f7096e67-1c66-4074-b306-32741be5ff9b"
-					(reference "#PWR01401")
+					(reference "#PWR1401")
 					(unit 1)
 				)
@@
 		(on_board yes)
 		(dnp no)
-		(property "Reference" "#PWR01428"
+		(property "Reference" "#PWR1428"
 			(at 166.37 146.05 0)
 			(effects
@@
 			(project "sax2"
 				(path "/6c8448b4-b04d-47e1-934e-e40cbe27a7be/f7096e67-1c66-4074-b306-32741be5ff9b"
-					(reference "#PWR01428")
+					(reference "#PWR1428")
 					(unit 1)
 				)
@@
 		(on_board yes)
 		(dnp no)
-		(property "Reference" "#PWR01415"
+		(property "Reference" "#PWR1415"
 			(at 138.43 97.79 0)
 			(effects
@@
 			(project "sax2"
 				(path "/6c8448b4-b04d-47e1-934e-e40cbe27a7be/f7096e67-1c66-4074-b306-32741be5ff9b"
-					(reference "#PWR01415")
+					(reference "#PWR1415")
 					(unit 1)
 				)
@@
 		(on_board yes)
 		(dnp no)
-		(property "Reference" "#PWR01420"
+		(property "Reference" "#PWR1420"
 			(at 214.63 106.68 0)
 			(effects
@@
 			(project "sax2"
 				(path "/6c8448b4-b04d-47e1-934e-e40cbe27a7be/f7096e67-1c66-4074-b306-32741be5ff9b"
-					(reference "#PWR01420")
-					(unit 1)
-				)
-			)
-		)
-	)
-	(symbol
-		(lib_id "V2_Device:C_0603_0u1")
+					(reference "#PWR1420")
+					(unit 1)
+				)
+			)
+		)
+	)
+	(symbol
+		(lib_id "V2_Capacitor:0603_0u1")
 		(at 213.36 93.98 0)
 		(unit 1)
@@
 		(on_board yes)
 		(dnp no)
-		(property "Reference" "#PWR01410"
+		(property "Reference" "#PWR1410"
 			(at 213.36 101.6 0)
 			(effects
@@
 			(project "sax2"
 				(path "/6c8448b4-b04d-47e1-934e-e40cbe27a7be/f7096e67-1c66-4074-b306-32741be5ff9b"
-					(reference "#PWR01410")
+					(reference "#PWR1410")
 					(unit 1)
 				)
@@
 		(on_board yes)
 		(dnp no)
-		(property "Reference" "#PWR01402"
+		(property "Reference" "#PWR1402"
 			(at 129.54 88.9 0)
 			(effects
@@
 			(project "sax2"
 				(path "/6c8448b4-b04d-47e1-934e-e40cbe27a7be/f7096e67-1c66-4074-b306-32741be5ff9b"
-					(reference "#PWR01402")
+					(reference "#PWR1402")
 					(unit 1)
 				)
@@
 		(on_board yes)
 		(dnp no)
-		(property "Reference" "#PWR01408"
+		(property "Reference" "#PWR1408"
 			(at 149.86 97.79 0)
 			(effects
@@
 			(project "sax2"
 				(path "/6c8448b4-b04d-47e1-934e-e40cbe27a7be/f7096e67-1c66-4074-b306-32741be5ff9b"
-					(reference "#PWR01408")
+					(reference "#PWR1408")
 					(unit 1)
 				)
@@
 	)
 	(symbol
-		(lib_id "V2_Device:C_0603_0u47")
+		(lib_id "V2_Capacitor:0603_0u47")
 		(at 129.54 97.79 90)
 		(unit 1)
@@
 		(on_board yes)
 		(dnp no)
-		(property "Reference" "#PWR01419"
+		(property "Reference" "#PWR1419"
 			(at 194.31 106.68 0)
 			(effects
@@
 			(project "sax2"
 				(path "/6c8448b4-b04d-47e1-934e-e40cbe27a7be/f7096e67-1c66-4074-b306-32741be5ff9b"
-					(reference "#PWR01419")
+					(reference "#PWR1419")
 					(unit 1)
 				)
@@
 		(on_board yes)
 		(dnp no)
-		(property "Reference" "#PWR01417"
+		(property "Reference" "#PWR1417"
 			(at 184.15 99.06 0)
 			(effects
@@
 			(project "sax2"
 				(path "/6c8448b4-b04d-47e1-934e-e40cbe27a7be/f7096e67-1c66-4074-b306-32741be5ff9b"
-					(reference "#PWR01417")
+					(reference "#PWR1417")
 					(unit 1)
 				)
@@
 		(on_board yes)
 		(dnp no)
-		(property "Reference" "#PWR01409"
+		(property "Reference" "#PWR1409"
 			(at 184.15 93.98 0)
 			(effects
@@
 			(project "sax2"
 				(path "/6c8448b4-b04d-47e1-934e-e40cbe27a7be/f7096e67-1c66-4074-b306-32741be5ff9b"
-					(reference "#PWR01409")
+					(reference "#PWR1409")
 					(unit 1)
 				)
@@
 		(on_board yes)
 		(dnp no)
-		(property "Reference" "#PWR01406"
+		(property "Reference" "#PWR1406"
 			(at 213.36 95.25 0)
 			(effects
@@
 			(project "sax2"
 				(path "/6c8448b4-b04d-47e1-934e-e40cbe27a7be/f7096e67-1c66-4074-b306-32741be5ff9b"
-					(reference "#PWR01406")
+					(reference "#PWR1406")
 					(unit 1)
 				)
@@
 		(on_board yes)
 		(dnp no)
-		(property "Reference" "#PWR01421"
+		(property "Reference" "#PWR1421"
 			(at 97.79 107.95 0)
 			(effects
@@
 			(project "sax2"
 				(path "/6c8448b4-b04d-47e1-934e-e40cbe27a7be/f7096e67-1c66-4074-b306-32741be5ff9b"
-					(reference "#PWR01421")
+					(reference "#PWR1421")
 					(unit 1)
 				)
@@
 	)
 	(symbol
-		(lib_id "V2_Device:R_0603_2k7")
+		(lib_id "V2_Resistor:0603_2k7")
 		(at 151.13 96.52 0)
 		(unit 1)
@@
 		(on_board yes)
 		(dnp no)
-		(property "Reference" "#PWR01427"
+		(property "Reference" "#PWR1427"
 			(at 156.21 140.97 0)
 			(effects
@@
 			(project "sax2"
 				(path "/6c8448b4-b04d-47e1-934e-e40cbe27a7be/f7096e67-1c66-4074-b306-32741be5ff9b"
-					(reference "#PWR01427")
+					(reference "#PWR1427")
 					(unit 1)
 				)
@@
 		(on_board yes)
 		(dnp no)
-		(property "Reference" "#PWR01422"
+		(property "Reference" "#PWR1422"
 			(at 130.81 113.03 0)
 			(effects
@@
 			(project "sax2"
 				(path "/6c8448b4-b04d-47e1-934e-e40cbe27a7be/f7096e67-1c66-4074-b306-32741be5ff9b"
-					(reference "#PWR01422")
-					(unit 1)
-				)
+					(reference "#PWR1422")
+					(unit 1)
+				)

Commit message: Update
Changed lines of the file:
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@@
 		)
 		(property "Value" "+3V3"
-			(at 93.98 80.01 0)
-			(effects
-				(font
-					(size 1.27 1.27)
+			(at 93.98 79.502 0)
+			(effects
+				(font
+					(size 1.27 1.27)
+					(color 255 92 187 1)
 				)
 			)
@@
 		)
 		(property "Value" "+3V3"
-			(at 124.46 73.66 0)
-			(effects
-				(font
-					(size 1.27 1.27)
+			(at 124.46 73.152 0)
+			(effects
+				(font
+					(size 1.27 1.27)
+					(color 255 92 187 1)
 				)
 			)
@@
 		)
 		(property "Value" "+3V3"
-			(at 149.86 90.17 0)
-			(effects
-				(font
-					(size 1.27 1.27)
+			(at 149.86 89.662 0)
+			(effects
+				(font
+					(size 1.27 1.27)
+					(color 255 92 187 1)
 				)
 			)
@@
 		)
 		(property "Value" "+3V3"
-			(at 184.15 106.045 90)
-			(effects
-				(font
-					(size 1.27 1.27)
+			(at 184.15 106.045 0)
+			(effects
+				(font
+					(size 1.27 1.27)
+					(color 255 92 187 1)
 				)
 			)
@@
 				(font
 					(size 1.27 1.27)
+					(color 255 92 187 1)
 				)
 			)
@@
 		)
 		(property "Value" "+5V"
-			(at 167.132 140.97 90)
-			(effects
-				(font
-					(size 1.27 1.27)
-				)
-				(justify right)
-			)
-		)
+			(at 165.608 140.97 90)
+			(effects
+				(font
+					(size 1.27 1.27)
+					(color 255 92 187 1)
+				)
+			)
+		)
