File: hardware/sax2/PressureSensor.kicad_sch (KiCad schematic)
At the start: 5 parts, among them IC1401 MP3V5004GP

Commit message: Update library
Parts:
- C1402: Rating (none) -> 50V
Changed lines of the file:
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@@
 			)
 		)
-		(property "Description" "Power symbol creates a global label with name \"GND\" , ground"
+		(property "Description" ""
 			(at 125.73 93.98 0)
 			(effects
@@
 			)
 		)
-		(property "Description" "Power symbol creates a global label with name \"+3V3\""
+		(property "Description" ""
 			(at 125.73 88.9 0)
 			(effects
@@
 			)
 		)
-		(property "Description" "Power symbol creates a global label with name \"+3V3\""
+		(property "Description" ""
 			(at 156.21 86.36 0)
 			(effects
@@
 			)
 		)
-		(property "Description" "Power symbol creates a global label with name \"GND\" , ground"
+		(property "Description" ""
 			(at 177.8 96.52 0)
 			(effects
@@
 		(property "Product" "CGA3E2X7R1H104M080AA"
 			(at 125.73 109.22 0)
+			(effects
+				(font
+					(size 1.27 1.27)
+				)
+				(hide yes)
+			)
+		)
+		(property "Rating" "50V"
+			(at 125.73 114.3 0)
 			(effects
 				(font
@@
 			)
 		)
-		(property "Description" "Power symbol creates a global label with name \"GND\" , ground"
+		(property "Description" ""
 			(at 165.1 96.52 0)
 			(effects
@@
 			)
 		)
-		(property "Description" "Power symbol creates a global label with name \"GND\" , ground"
+		(property "Description" ""
 			(at 156.21 96.52 0)
 			(effects
@@
 			)
 		)
-		(property "Description" "Power symbol creates a global label with name \"+5V\""
+		(property "Description" ""
 			(at 161.29 127 0)
 			(effects
@@
 			)
 		)
-		(property "Description" "Power symbol creates a global label with name \"GND\" , ground"
+		(property "Description" ""
 			(at 161.29 132.08 0)
 			(effects

Commit message: Update Library
Parts:
- C1402: symbol V2_Device:C_0603_0u1 -> V2_Capacitor:0603_0u1
- C1403: symbol V2_Device:C_0603_0u022 -> V2_Capacitor:0603_0u022
- R1404: symbol V2_Device:R_0603_100k -> V2_Resistor:0603_100k
Changed lines of the file:
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@@
 	)
 	(symbol
-		(lib_id "V2_Device:C_0603_0u022")
+		(lib_id "V2_Capacitor:0603_0u022")
 		(at 165.1 93.98 0)
 		(unit 1)
@@
 		(dnp no)
 		(fields_autoplaced yes)
-		(property "Reference" "#PWR01407"
+		(property "Reference" "#PWR1407"
 			(at 125.73 100.33 0)
 			(effects
@@
 			(project "sax2"
 				(path "/6c8448b4-b04d-47e1-934e-e40cbe27a7be/6178bc16-76cb-41ae-a61c-619a3590ea5a"
-					(reference "#PWR01407")
+					(reference "#PWR1407")
 					(unit 1)
 				)
@@
 		(on_board yes)
 		(dnp no)
-		(property "Reference" "#PWR01405"
+		(property "Reference" "#PWR1405"
 			(at 125.73 92.71 0)
 			(effects
@@
 			(project "sax2"
 				(path "/6c8448b4-b04d-47e1-934e-e40cbe27a7be/6178bc16-76cb-41ae-a61c-619a3590ea5a"
-					(reference "#PWR01405")
+					(reference "#PWR1405")
 					(unit 1)
 				)
@@
 		(on_board yes)
 		(dnp no)
-		(property "Reference" "#PWR01404"
+		(property "Reference" "#PWR1404"
 			(at 152.4 86.36 0)
 			(effects
@@
 			(project "sax2"
 				(path "/6c8448b4-b04d-47e1-934e-e40cbe27a7be/6178bc16-76cb-41ae-a61c-619a3590ea5a"
-					(reference "#PWR01404")
+					(reference "#PWR1404")
 					(unit 1)
 				)
@@
 		(dnp no)
 		(fields_autoplaced yes)
-		(property "Reference" "#PWR01413"
+		(property "Reference" "#PWR1413"
 			(at 177.8 102.87 0)
 			(effects
@@
 			(project "sax2"
 				(path "/6c8448b4-b04d-47e1-934e-e40cbe27a7be/6178bc16-76cb-41ae-a61c-619a3590ea5a"
-					(reference "#PWR01413")
-					(unit 1)
-				)
-			)
-		)
-	)
-	(symbol
-		(lib_id "V2_Device:C_0603_0u1")
+					(reference "#PWR1413")
+					(unit 1)
+				)
+			)
+		)
+	)
+	(symbol
+		(lib_id "V2_Capacitor:0603_0u1")
 		(at 125.73 91.44 0)
 		(unit 1)
@@
 		(dnp no)
 		(fields_autoplaced yes)
-		(property "Reference" "#PWR01412"
+		(property "Reference" "#PWR1412"
 			(at 165.1 102.87 0)
 			(effects
@@
 			(project "sax2"
 				(path "/6c8448b4-b04d-47e1-934e-e40cbe27a7be/6178bc16-76cb-41ae-a61c-619a3590ea5a"
-					(reference "#PWR01412")
+					(reference "#PWR1412")
 					(unit 1)
 				)
@@
 		(dnp no)
 		(fields_autoplaced yes)
-		(property "Reference" "#PWR01411"
+		(property "Reference" "#PWR1411"
 			(at 162.56 96.52 0)
 			(effects
@@
 			(project "sax2"
 				(path "/6c8448b4-b04d-47e1-934e-e40cbe27a7be/6178bc16-76cb-41ae-a61c-619a3590ea5a"
-					(reference "#PWR01411")
+					(reference "#PWR1411")
 					(unit 1)
 				)
@@
 		(on_board yes)
 		(dnp no)
-		(property "Reference" "#PWR01424"
+		(property "Reference" "#PWR1424"
 			(at 157.48 127 0)
 			(effects
@@
 			(project "sax2"
 				(path "/6c8448b4-b04d-47e1-934e-e40cbe27a7be/6178bc16-76cb-41ae-a61c-619a3590ea5a"
-					(reference "#PWR01424")
+					(reference "#PWR1424")
 					(unit 1)
 				)
@@
 	)
 	(symbol
-		(lib_id "V2_Device:R_0603_100k")
+		(lib_id "V2_Resistor:0603_100k")
 		(at 177.8 93.98 0)
 		(unit 1)
@@
 		(on_board yes)
 		(dnp no)
-		(property "Reference" "#PWR01426"
+		(property "Reference" "#PWR1426"
 			(at 167.64 132.08 0)
 			(effects
@@
 			(project "sax2"
 				(path "/6c8448b4-b04d-47e1-934e-e40cbe27a7be/6178bc16-76cb-41ae-a61c-619a3590ea5a"
-					(reference "#PWR01426")
-					(unit 1)
-				)
+					(reference "#PWR1426")
+					(unit 1)
+				)

Commit message: Update
Changed lines of the file:
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@@
 		)
 		(property "Value" "+3V3"
-			(at 123.444 83.566 0)
-			(effects
-				(font
-					(size 1.27 1.27)
-				)
-				(justify left)
+			(at 125.73 84.074 0)
+			(effects
+				(font
+					(size 1.27 1.27)
+					(color 255 92 187 1)
+				)
 			)
 		)
@@
 		)
 		(property "Value" "+3V3"
-			(at 160.02 86.36 90)
-			(effects
-				(font
-					(size 1.27 1.27)
-				)
-				(justify left)
+			(at 162.56 86.36 90)
+			(effects
+				(font
+					(size 1.27 1.27)
+					(color 255 92 187 1)
+				)
 			)
 		)
@@
 		)
 		(property "Value" "+5V"
-			(at 168.402 127 90)
-			(effects
-				(font
-					(size 1.27 1.27)
-				)
-				(justify right)
-			)
-		)
+			(at 167.64 127 90)
+			(effects
+				(font
+					(size 1.27 1.27)
+					(color 255 92 187 1)
+				)
+			)
+		)
