File: hardware/sax/AnalogSensors.kicad_sch (KiCad schematic)
At the start: 2 parts, among them J1301 2x05_Horizontal

Commit message: Update library
Parts:
- J1301: Manufacturer (none) -> Amphenol FCI; Mouser (none) -> 649-200211120001T4LF; Product (none) -> 20021112-00010T4LF
- TVS1301: footprint Diode_SMD:D_0603_1608Metric -> V2_Diode_SMD:D_0603; Manufacturer (none) -> Bourns; Mouser (none) -> 652-CG0603MLC-3.3LE; Product (none) -> CG0603MLC-3.3LE; Rating (none) -> 3V3
Changed lines of the file:
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@@
 			)
 		)
-		(property "Datasheet" "~"
+		(property "Datasheet" ""
 			(at 120.65 110.49 0)
 			(effects
@@
 			)
 		)
-		(property "Description" ""
+		(property "Description" "Amphenol – Minitek127"
 			(at 121.92 110.49 0)
 			(effects
@@
 			)
 		)
-		(property "Sim.Enable" "0"
-			(at 121.92 110.49 0)
+		(property "Mouser" "649-200211120001T4LF"
+			(at 121.92 133.35 0)
+			(effects
+				(font
+					(size 1.27 1.27)
+				)
+				(hide yes)
+			)
+		)
+		(property "Manufacturer" "Amphenol FCI"
+			(at 121.92 128.27 0)
+			(effects
+				(font
+					(size 1.27 1.27)
+				)
+				(hide yes)
+			)
+		)
+		(property "Product" "20021112-00010T4LF"
+			(at 121.92 130.81 0)
 			(effects
 				(font
@@
 	)
 	(symbol
-		(lib_id "power:+3V3")
+		(lib_id "V2_power:+3V3")
 		(at 128.27 115.57 270)
 		(unit 1)
@@
 			)
 		)
-		(property "Footprint" "Diode_SMD:D_0603_1608Metric"
+		(property "Footprint" "V2_Diode_SMD:D_0603"
 			(at 116.205 133.35 0)
 			(effects
@@
 			)
 		)
+		(property "Mouser" "652-CG0603MLC-3.3LE"
+			(at 128.27 133.35 0)
+			(effects
+				(font
+					(size 1.27 1.27)
+				)
+				(hide yes)
+			)
+		)
+		(property "Product" "CG0603MLC-3.3LE"
+			(at 123.19 133.35 0)
+			(effects
+				(font
+					(size 1.27 1.27)
+				)
+				(hide yes)
+			)
+		)
+		(property "Manufacturer" "Bourns"
+			(at 120.65 133.35 0)
+			(effects
+				(font
+					(size 1.27 1.27)
+				)
+				(hide yes)
+			)
+		)
+		(property "Rating" "3V3"
+			(at 125.73 133.35 0)
+			(effects
+				(font
+					(size 1.27 1.27)
+				)
+				(hide yes)
+			)
+		)
 		(pin "1"
 		)
@@
 	)
 	(symbol
-		(lib_id "power:GND")
+		(lib_id "V2_power:GND")
 		(at 110.49 137.16 0)
 		(mirror y)
@@
 	)
 	(symbol
-		(lib_id "power:GND")
+		(lib_id "V2_power:GND")
 		(at 115.57 115.57 270)
 		(unit 1)
@@
 	)
 	(symbol
-		(lib_id "power:+3V3")
+		(lib_id "V2_power:+3V3")
 		(at 110.49 129.54 0)
 		(mirror y)
