File: hardware/sax/ExpressionInput.kicad_sch (KiCad schematic)
At the start: 5 parts

Commit message: Update library
Parts:
- C1402: footprint Capacitor_SMD:C_0603_1608Metric -> V2_Capacitor_SMD:C_0603; symbol Device:C_Small -> V2_Device:C_0603_0u022; Manufacturer (none) -> YAGEO; Mouser (none) -> 603-CC603KPX7R9BB223; Product (none) -> CC0603KPX7R9BB223
- D1401: LCSC (none) -> C965555; Manufacturer (none) -> Worldsemi; Product (none) -> WS2812B-2020
- R1401: footprint Resistor_SMD:R_0603_1608Metric -> V2_Resistor_SMD:R_0603; symbol Device:R_Small -> V2_Device:R_0603_1k; Manufacturer (none) -> Vishay; Mouser (none) -> 71-CRCW06031K00FKEAH; Product (none) -> CRCW06031K00FKEAHP; Rating (none) -> 330mW
- R1404: footprint Resistor_SMD:R_0603_1608Metric -> V2_Resistor_SMD:R_0603; symbol Device:R_Small -> V2_Device:R_0603_100k; Manufacturer (none) -> Vishay; Mouser (none) -> 71-CRCW0603100KFKEAC; Product (none) -> CRCW0603100KFKEAC; Rating (none) -> 100mW
- TVS1401: footprint Diode_SMD:D_0603_1608Metric -> V2_Diode_SMD:D_0603; Manufacturer (none) -> Bourns; Mouser (none) -> 652-CG0603MLC-3.3LE; Product (none) -> CG0603MLC-3.3LE; Rating (none) -> 3V3
Changed lines of the file:
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@@
 	)
 	(symbol
-		(lib_id "Device:R_Small")
+		(lib_id "V2_Device:R_0603_1k")
 		(at 137.16 92.71 270)
 		(unit 1)
@@
 			)
 		)
-		(property "Footprint" "Resistor_SMD:R_0603_1608Metric"
+		(property "Footprint" "V2_Resistor_SMD:R_0603"
+			(at 121.412 92.71 0)
+			(effects
+				(font
+					(size 1.27 1.27)
+				)
+				(hide yes)
+			)
+		)
+		(property "Datasheet" ""
 			(at 137.16 92.71 0)
 			(effects
@@
 			)
 		)
-		(property "Datasheet" "~"
-			(at 137.16 92.71 0)
-			(effects
-				(font
-					(size 1.27 1.27)
-				)
-				(hide yes)
-			)
-		)
 		(property "Description" "Resistor, small symbol"
-			(at 137.16 92.71 0)
+			(at 121.92 92.71 0)
+			(effects
+				(font
+					(size 1.27 1.27)
+				)
+				(hide yes)
+			)
+		)
+		(property "Mouser" "71-CRCW06031K00FKEAH"
+			(at 111.76 92.71 0)
+			(effects
+				(font
+					(size 1.27 1.27)
+				)
+				(hide yes)
+			)
+		)
+		(property "Product" "CRCW06031K00FKEAHP"
+			(at 116.84 92.71 0)
+			(effects
+				(font
+					(size 1.27 1.27)
+				)
+				(hide yes)
+			)
+		)
+		(property "Manufacturer" "Vishay"
+			(at 119.38 92.71 0)
+			(effects
+				(font
+					(size 1.27 1.27)
+				)
+				(hide yes)
+			)
+		)
+		(property "Rating" "330mW"
+			(at 114.3 92.71 0)
 			(effects
 				(font
@@
 	)
 	(symbol
-		(lib_id "power:GND")
+		(lib_id "V2_power:GND")
 		(at 123.19 97.79 0)
 		(unit 1)
@@
 	)
 	(symbol
-		(lib_id "power:+5V")
+		(lib_id "V2_power:+5V")
 		(at 160.02 125.73 270)
 		(unit 1)
@@
 	)
 	(symbol
-		(lib_id "power:GND")
+		(lib_id "V2_power:GND")
 		(at 180.34 97.79 0)
 		(unit 1)
@@
 	)
 	(symbol
-		(lib_id "Device:C_Small")
+		(lib_id "V2_Device:C_0603_0u022")
 		(at 180.34 95.25 0)
 		(unit 1)
@@
 			)
 		)
-		(property "Footprint" "Capacitor_SMD:C_0603_1608Metric"
+		(property "Footprint" "V2_Capacitor_SMD:C_0603"
+			(at 180.34 112.268 0)
+			(effects
+				(font
+					(size 1.27 1.27)
+				)
+				(hide yes)
+			)
+		)
+		(property "Datasheet" ""
 			(at 180.34 95.25 0)
 			(effects
@@
 			)
 		)
-		(property "Datasheet" "~"
-			(at 180.34 95.25 0)
-			(effects
-				(font
-					(size 1.27 1.27)
-				)
-				(hide yes)
-			)
-		)
 		(property "Description" "Unpolarized capacitor, small symbol"
-			(at 180.34 95.25 0)
+			(at 180.34 107.95 0)
+			(effects
+				(font
+					(size 1.27 1.27)
+				)
+				(hide yes)
+			)
+		)
+		(property "Mouser" "603-CC603KPX7R9BB223"
+			(at 180.34 115.57 0)
+			(effects
+				(font
+					(size 1.27 1.27)
+				)
+				(hide yes)
+			)
+		)
+		(property "Product" "CC0603KPX7R9BB223"
+			(at 180.34 113.03 0)
+			(effects
+				(font
+					(size 1.27 1.27)
+				)
+				(hide yes)
+			)
+		)
+		(property "Manufacturer" "YAGEO"
+			(at 180.34 110.49 0)
 			(effects
 				(font
@@
 			)
 		)
-		(property "Footprint" "Diode_SMD:D_0603_1608Metric"
+		(property "Footprint" "V2_Diode_SMD:D_0603"
 			(at 154.305 96.52 0)
 			(effects
@@
 		(property "Description" ""
 			(at 148.59 96.52 0)
+			(effects
+				(font
+					(size 1.27 1.27)
+				)
+				(hide yes)
+			)
+		)
+		(property "Mouser" "652-CG0603MLC-3.3LE"
+			(at 166.37 96.52 0)
+			(effects
+				(font
+					(size 1.27 1.27)
+				)
+				(hide yes)
+			)
+		)
+		(property "Product" "CG0603MLC-3.3LE"
+			(at 161.29 96.52 0)
+			(effects
+				(font
+					(size 1.27 1.27)
+				)
+				(hide yes)
+			)
+		)
+		(property "Manufacturer" "Bourns"
+			(at 158.75 96.52 0)
+			(effects
+				(font
+					(size 1.27 1.27)
+				)
+				(hide yes)
+			)
+		)
+		(property "Rating" "3V3"
+			(at 163.83 96.52 0)
 			(effects
 				(font
@@
 	)
 	(symbol
-		(lib_id "power:GND")
+		(lib_id "V2_power:GND")
 		(at 160.02 130.81 90)
 		(unit 1)
@@
 	)
 	(symbol
-		(lib_id "power:GND")
+		(lib_id "V2_power:GND")
 		(at 148.59 100.33 0)
 		(unit 1)
@@
 			)
 		)
+		(property "Manufacturer" "Worldsemi"
+			(at 152.4 145.034 0)
+			(effects
+				(font
+					(size 1.27 1.27)
+				)
+				(hide yes)
+			)
+		)
+		(property "Product" "WS2812B-2020"
+			(at 152.4 142.494 0)
+			(effects
+				(font
+					(size 1.27 1.27)
+				)
+				(hide yes)
+			)
+		)
+		(property "LCSC" "C965555"
+			(at 152.4 147.828 0)
+			(effects
+				(font
+					(size 1.27 1.27)
+				)
+				(hide yes)
+			)
+		)
 		(pin "1"
 		)
@@
 	)
 	(symbol
-		(lib_id "Device:R_Small")
+		(lib_id "V2_Device:R_0603_100k")
 		(at 123.19 95.25 0)
 		(unit 1)
@@
 			)
 		)
-		(property "Footprint" "Resistor_SMD:R_0603_1608Metric"
+		(property "Footprint" "V2_Resistor_SMD:R_0603"
+			(at 123.19 110.998 0)
+			(effects
+				(font
+					(size 1.27 1.27)
+				)
+				(hide yes)
+			)
+		)
+		(property "Datasheet" ""
 			(at 123.19 95.25 0)
 			(effects
@@
 			)
 		)
-		(property "Datasheet" "~"
-			(at 123.19 95.25 0)
-			(effects
-				(font
-					(size 1.27 1.27)
-				)
-				(hide yes)
-			)
-		)
 		(property "Description" "Resistor, small symbol"
-			(at 123.19 95.25 0)
-			(effects
-				(font
+			(at 123.19 107.95 0)
+			(effects
+				(font
+					(size 1.27 1.27)
+				)
+				(hide yes)
+			)
+		)
+		(property "Mouser" "71-CRCW0603100KFKEAC"
+			(at 123.19 118.11 0)
+			(effects
+				(font
+					(size 1.27 1.27)
+				)
+				(hide yes)
+			)
+		)
+		(property "Rating" "100mW"
+			(at 123.19 115.57 0)
+			(effects
+				(font
+					(size 1.27 1.27)
+				)
+				(hide yes)
+			)
+		)
+		(property "Manufacturer" "Vishay"
+			(at 123.19 110.49 0)
+			(effects
+				(font
+					(size 1.27 1.27)
+				)
+				(hide yes)
+			)
+		)
+		(property "Product" "CRCW0603100KFKEAC"
+			(at 123.19 113.03 0)
+			(effects
+				(font

Commit message: Update Library
Parts:
- C1402: symbol V2_Device:C_0603_0u022 -> V2_Capacitor:0603_0u022
- R1401: symbol V2_Device:R_0603_1k -> V2_Resistor:0603_1k
- R1404: symbol V2_Device:R_0603_100k -> V2_Resistor:0603_100k
Changed lines of the file:
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@@
 	)
 	(symbol
-		(lib_id "V2_Device:R_0603_1k")
+		(lib_id "V2_Resistor:0603_1k")
 		(at 137.16 92.71 270)
 		(unit 1)
@@
 		(dnp no)
 		(fields_autoplaced yes)
-		(property "Reference" "#PWR01404"
+		(property "Reference" "#PWR1404"
 			(at 123.19 104.14 0)
 			(effects
@@
 			(project "sax"
 				(path "/6c8448b4-b04d-47e1-934e-e40cbe27a7be/986c2710-b6fb-48af-9291-0e7dc7b5abf9/09fde53a-0726-4a1a-ba32-997a9c8cb2ac"
-					(reference "#PWR01701")
+					(reference "#PWR1701")
 					(unit 1)
 				)
 				(path "/6c8448b4-b04d-47e1-934e-e40cbe27a7be/986c2710-b6fb-48af-9291-0e7dc7b5abf9/75bdefb6-cbec-430c-b2f6-bba8982a1e16"
-					(reference "#PWR01404")
+					(reference "#PWR1404")
 					(unit 1)
 				)
 				(path "/6c8448b4-b04d-47e1-934e-e40cbe27a7be/986c2710-b6fb-48af-9291-0e7dc7b5abf9/7eddc4ac-e264-4e8d-993d-81fc85f367c8"
-					(reference "#PWR01501")
+					(reference "#PWR1501")
 					(unit 1)
 				)
 				(path "/6c8448b4-b04d-47e1-934e-e40cbe27a7be/986c2710-b6fb-48af-9291-0e7dc7b5abf9/ab1436ac-5052-4cae-b140-374128cd8279"
-					(reference "#PWR02101")
+					(reference "#PWR2101")
 					(unit 1)
 				)
 				(path "/6c8448b4-b04d-47e1-934e-e40cbe27a7be/986c2710-b6fb-48af-9291-0e7dc7b5abf9/b1b709ba-4565-4658-b8d7-ca720ae6b4d0"
-					(reference "#PWR01901")
+					(reference "#PWR1901")
 					(unit 1)
 				)
 				(path "/6c8448b4-b04d-47e1-934e-e40cbe27a7be/986c2710-b6fb-48af-9291-0e7dc7b5abf9/e5e66090-238e-4b5d-8478-8d0716aa9aa6"
-					(reference "#PWR01601")
+					(reference "#PWR1601")
 					(unit 1)
 				)
 				(path "/6c8448b4-b04d-47e1-934e-e40cbe27a7be/986c2710-b6fb-48af-9291-0e7dc7b5abf9/f153ee55-65c6-4eb1-a6b0-fdf78a9680f1"
-					(reference "#PWR02001")
+					(reference "#PWR2001")
 					(unit 1)
 				)
 				(path "/6c8448b4-b04d-47e1-934e-e40cbe27a7be/986c2710-b6fb-48af-9291-0e7dc7b5abf9/f5d1679c-7076-43d7-b0e0-c560820060c0"
-					(reference "#PWR01801")
+					(reference "#PWR1801")
 					(unit 1)
 				)
@@
 		(dnp no)
 		(fields_autoplaced yes)
-		(property "Reference" "#PWR01417"
+		(property "Reference" "#PWR1417"
 			(at 156.21 125.73 0)
 			(effects
@@
 			(project "sax"
 				(path "/6c8448b4-b04d-47e1-934e-e40cbe27a7be/986c2710-b6fb-48af-9291-0e7dc7b5abf9/09fde53a-0726-4a1a-ba32-997a9c8cb2ac"
-					(reference "#PWR01704")
+					(reference "#PWR1704")
 					(unit 1)
 				)
 				(path "/6c8448b4-b04d-47e1-934e-e40cbe27a7be/986c2710-b6fb-48af-9291-0e7dc7b5abf9/75bdefb6-cbec-430c-b2f6-bba8982a1e16"
-					(reference "#PWR01417")
+					(reference "#PWR1417")
 					(unit 1)
 				)
 				(path "/6c8448b4-b04d-47e1-934e-e40cbe27a7be/986c2710-b6fb-48af-9291-0e7dc7b5abf9/7eddc4ac-e264-4e8d-993d-81fc85f367c8"
-					(reference "#PWR01504")
+					(reference "#PWR1504")
 					(unit 1)
 				)
 				(path "/6c8448b4-b04d-47e1-934e-e40cbe27a7be/986c2710-b6fb-48af-9291-0e7dc7b5abf9/ab1436ac-5052-4cae-b140-374128cd8279"
-					(reference "#PWR02104")
+					(reference "#PWR2104")
 					(unit 1)
 				)
 				(path "/6c8448b4-b04d-47e1-934e-e40cbe27a7be/986c2710-b6fb-48af-9291-0e7dc7b5abf9/b1b709ba-4565-4658-b8d7-ca720ae6b4d0"
-					(reference "#PWR01904")
+					(reference "#PWR1904")
 					(unit 1)
 				)
 				(path "/6c8448b4-b04d-47e1-934e-e40cbe27a7be/986c2710-b6fb-48af-9291-0e7dc7b5abf9/e5e66090-238e-4b5d-8478-8d0716aa9aa6"
-					(reference "#PWR01604")
+					(reference "#PWR1604")
 					(unit 1)
 				)
 				(path "/6c8448b4-b04d-47e1-934e-e40cbe27a7be/986c2710-b6fb-48af-9291-0e7dc7b5abf9/f153ee55-65c6-4eb1-a6b0-fdf78a9680f1"
-					(reference "#PWR02004")
+					(reference "#PWR2004")
 					(unit 1)
 				)
 				(path "/6c8448b4-b04d-47e1-934e-e40cbe27a7be/986c2710-b6fb-48af-9291-0e7dc7b5abf9/f5d1679c-7076-43d7-b0e0-c560820060c0"
-					(reference "#PWR01804")
+					(reference "#PWR1804")
 					(unit 1)
 				)
@@
 		(dnp no)
 		(fields_autoplaced yes)
-		(property "Reference" "#PWR01405"
+		(property "Reference" "#PWR1405"
 			(at 180.34 104.14 0)
 			(effects
@@
 			(project "sax"
 				(path "/6c8448b4-b04d-47e1-934e-e40cbe27a7be/986c2710-b6fb-48af-9291-0e7dc7b5abf9/09fde53a-0726-4a1a-ba32-997a9c8cb2ac"
-					(reference "#PWR01702")
+					(reference "#PWR1702")
 					(unit 1)
 				)
 				(path "/6c8448b4-b04d-47e1-934e-e40cbe27a7be/986c2710-b6fb-48af-9291-0e7dc7b5abf9/75bdefb6-cbec-430c-b2f6-bba8982a1e16"
-					(reference "#PWR01405")
+					(reference "#PWR1405")
 					(unit 1)
 				)
 				(path "/6c8448b4-b04d-47e1-934e-e40cbe27a7be/986c2710-b6fb-48af-9291-0e7dc7b5abf9/7eddc4ac-e264-4e8d-993d-81fc85f367c8"
-					(reference "#PWR01502")
+					(reference "#PWR1502")
 					(unit 1)
 				)
 				(path "/6c8448b4-b04d-47e1-934e-e40cbe27a7be/986c2710-b6fb-48af-9291-0e7dc7b5abf9/ab1436ac-5052-4cae-b140-374128cd8279"
-					(reference "#PWR02102")
+					(reference "#PWR2102")
 					(unit 1)
 				)
 				(path "/6c8448b4-b04d-47e1-934e-e40cbe27a7be/986c2710-b6fb-48af-9291-0e7dc7b5abf9/b1b709ba-4565-4658-b8d7-ca720ae6b4d0"
-					(reference "#PWR01902")
+					(reference "#PWR1902")
 					(unit 1)
 				)
 				(path "/6c8448b4-b04d-47e1-934e-e40cbe27a7be/986c2710-b6fb-48af-9291-0e7dc7b5abf9/e5e66090-238e-4b5d-8478-8d0716aa9aa6"
-					(reference "#PWR01602")
+					(reference "#PWR1602")
 					(unit 1)
 				)
 				(path "/6c8448b4-b04d-47e1-934e-e40cbe27a7be/986c2710-b6fb-48af-9291-0e7dc7b5abf9/f153ee55-65c6-4eb1-a6b0-fdf78a9680f1"
-					(reference "#PWR02002")
+					(reference "#PWR2002")
 					(unit 1)
 				)
 				(path "/6c8448b4-b04d-47e1-934e-e40cbe27a7be/986c2710-b6fb-48af-9291-0e7dc7b5abf9/f5d1679c-7076-43d7-b0e0-c560820060c0"
-					(reference "#PWR01802")
+					(reference "#PWR1802")
 					(unit 1)
 				)
@@
 	)
 	(symbol
-		(lib_id "V2_Device:C_0603_0u022")
+		(lib_id "V2_Capacitor:0603_0u022")
 		(at 180.34 95.25 0)
 		(unit 1)
@@
 		(dnp no)
 		(fields_autoplaced yes)
-		(property "Reference" "#PWR01418"
+		(property "Reference" "#PWR1418"
 			(at 166.37 130.81 0)
 			(effects
@@
 			(project "sax"
 				(path "/6c8448b4-b04d-47e1-934e-e40cbe27a7be/986c2710-b6fb-48af-9291-0e7dc7b5abf9/09fde53a-0726-4a1a-ba32-997a9c8cb2ac"
-					(reference "#PWR01705")
+					(reference "#PWR1705")
 					(unit 1)
 				)
 				(path "/6c8448b4-b04d-47e1-934e-e40cbe27a7be/986c2710-b6fb-48af-9291-0e7dc7b5abf9/75bdefb6-cbec-430c-b2f6-bba8982a1e16"
-					(reference "#PWR01418")
+					(reference "#PWR1418")
 					(unit 1)
 				)
 				(path "/6c8448b4-b04d-47e1-934e-e40cbe27a7be/986c2710-b6fb-48af-9291-0e7dc7b5abf9/7eddc4ac-e264-4e8d-993d-81fc85f367c8"
-					(reference "#PWR01505")
+					(reference "#PWR1505")
 					(unit 1)
 				)
 				(path "/6c8448b4-b04d-47e1-934e-e40cbe27a7be/986c2710-b6fb-48af-9291-0e7dc7b5abf9/ab1436ac-5052-4cae-b140-374128cd8279"
-					(reference "#PWR02105")
+					(reference "#PWR2105")
 					(unit 1)
 				)
 				(path "/6c8448b4-b04d-47e1-934e-e40cbe27a7be/986c2710-b6fb-48af-9291-0e7dc7b5abf9/b1b709ba-4565-4658-b8d7-ca720ae6b4d0"
-					(reference "#PWR01905")
+					(reference "#PWR1905")
 					(unit 1)
 				)
 				(path "/6c8448b4-b04d-47e1-934e-e40cbe27a7be/986c2710-b6fb-48af-9291-0e7dc7b5abf9/e5e66090-238e-4b5d-8478-8d0716aa9aa6"
-					(reference "#PWR01605")
+					(reference "#PWR1605")
 					(unit 1)
 				)
 				(path "/6c8448b4-b04d-47e1-934e-e40cbe27a7be/986c2710-b6fb-48af-9291-0e7dc7b5abf9/f153ee55-65c6-4eb1-a6b0-fdf78a9680f1"
-					(reference "#PWR02005")
+					(reference "#PWR2005")
 					(unit 1)
 				)
 				(path "/6c8448b4-b04d-47e1-934e-e40cbe27a7be/986c2710-b6fb-48af-9291-0e7dc7b5abf9/f5d1679c-7076-43d7-b0e0-c560820060c0"
-					(reference "#PWR01805")
+					(reference "#PWR1805")
 					(unit 1)
 				)
@@
 		(dnp no)
 		(fields_autoplaced yes)
-		(property "Reference" "#PWR01407"
+		(property "Reference" "#PWR1407"
 			(at 148.59 106.68 0)
 			(effects
@@
 			(project "sax"
 				(path "/6c8448b4-b04d-47e1-934e-e40cbe27a7be/986c2710-b6fb-48af-9291-0e7dc7b5abf9/09fde53a-0726-4a1a-ba32-997a9c8cb2ac"
-					(reference "#PWR01703")
+					(reference "#PWR1703")
 					(unit 1)
 				)
 				(path "/6c8448b4-b04d-47e1-934e-e40cbe27a7be/986c2710-b6fb-48af-9291-0e7dc7b5abf9/75bdefb6-cbec-430c-b2f6-bba8982a1e16"
-					(reference "#PWR01407")
+					(reference "#PWR1407")
 					(unit 1)
 				)
 				(path "/6c8448b4-b04d-47e1-934e-e40cbe27a7be/986c2710-b6fb-48af-9291-0e7dc7b5abf9/7eddc4ac-e264-4e8d-993d-81fc85f367c8"
-					(reference "#PWR01503")
+					(reference "#PWR1503")
 					(unit 1)
 				)
 				(path "/6c8448b4-b04d-47e1-934e-e40cbe27a7be/986c2710-b6fb-48af-9291-0e7dc7b5abf9/ab1436ac-5052-4cae-b140-374128cd8279"
-					(reference "#PWR02103")
+					(reference "#PWR2103")
 					(unit 1)
 				)
 				(path "/6c8448b4-b04d-47e1-934e-e40cbe27a7be/986c2710-b6fb-48af-9291-0e7dc7b5abf9/b1b709ba-4565-4658-b8d7-ca720ae6b4d0"
-					(reference "#PWR01903")
+					(reference "#PWR1903")
 					(unit 1)
 				)
 				(path "/6c8448b4-b04d-47e1-934e-e40cbe27a7be/986c2710-b6fb-48af-9291-0e7dc7b5abf9/e5e66090-238e-4b5d-8478-8d0716aa9aa6"
-					(reference "#PWR01603")
+					(reference "#PWR1603")
 					(unit 1)
 				)
 				(path "/6c8448b4-b04d-47e1-934e-e40cbe27a7be/986c2710-b6fb-48af-9291-0e7dc7b5abf9/f153ee55-65c6-4eb1-a6b0-fdf78a9680f1"
-					(reference "#PWR02003")
+					(reference "#PWR2003")
 					(unit 1)
 				)
 				(path "/6c8448b4-b04d-47e1-934e-e40cbe27a7be/986c2710-b6fb-48af-9291-0e7dc7b5abf9/f5d1679c-7076-43d7-b0e0-c560820060c0"
-					(reference "#PWR01803")
+					(reference "#PWR1803")
 					(unit 1)
 				)
@@
 	)
 	(symbol
-		(lib_id "V2_Device:R_0603_100k")
+		(lib_id "V2_Resistor:0603_100k")
 		(at 123.19 95.25 0)
 		(unit 1)
