File: hardware/sax/ExpressionInput.kicad_sch (KiCad schematic)
At the start: 5 parts

Commit message: Update
Parts:
- renumbered R1405 to R1403, R1403 to R1404

Commit message: Good Bye Imperial
Parts:
- C1405: footprint V2_Capacitor_SMD:C_0603 -> V2_Capacitor_SMD:C_1608; symbol V2_Capacitor:0603_0u022 -> V2_Capacitor:1608_0u022
- R1403: footprint V2_Resistor_SMD:R_0603 -> V2_Resistor_SMD:R_1608; symbol V2_Resistor:0603_100k -> V2_Resistor:1608_100k
- R1404: footprint V2_Resistor_SMD:R_0603 -> V2_Resistor_SMD:R_1608; symbol V2_Resistor:0603_1k -> V2_Resistor:1608_1k
Changed lines of the file:
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@@
 	)
 	(symbol
-		(lib_id "V2_Resistor:0603_1k")
+		(lib_id "V2_Resistor:1608_1k")
 		(at 137.16 92.71 270)
 		(unit 1)
@@
 			)
 		)
-		(property "Footprint" "V2_Resistor_SMD:R_0603"
+		(property "Footprint" "V2_Resistor_SMD:R_1608"
 			(at 121.412 92.71 0)
 			(hide yes)
@@
 	)
 	(symbol
-		(lib_id "V2_Capacitor:0603_0u022")
+		(lib_id "V2_Capacitor:1608_0u022")
 		(at 180.34 95.25 0)
 		(unit 1)
@@
 			)
 		)
-		(property "Footprint" "V2_Capacitor_SMD:C_0603"
+		(property "Footprint" "V2_Capacitor_SMD:C_1608"
 			(at 180.34 112.268 0)
 			(hide yes)
@@
 	)
 	(symbol
-		(lib_id "V2_Resistor:0603_100k")
+		(lib_id "V2_Resistor:1608_100k")
 		(at 123.19 95.25 0)
 		(unit 1)
@@
 			)
 		)
-		(property "Footprint" "V2_Resistor_SMD:R_0603"
+		(property "Footprint" "V2_Resistor_SMD:R_1608"
 			(at 123.19 110.998 0)
 			(hide yes)

Commit message: Refresh
Parts:
- TVS501: renamed from TVS1401; footprint V2_Diode_SMD:D_0603 -> V2_Diode_SMD:D_1608
- renumbered C1405 to C501, D1401 to D501, R1403 to R501, R1404 to R502
