File: hardware/sax/LinkPlug.kicad_sch (KiCad schematic)
At the start: 4 parts, among them J1101 NE8FAH, U1101 THVD24x2

Commit message: Update library
Parts:
- C1101: footprint Capacitor_SMD:C_0603_1608Metric -> V2_Capacitor_SMD:C_0603; symbol Device:C_Small -> V2_Device:C_0603_0u1; Manufacturer (none) -> TDK; Mouser (none) -> 810-CGA3E2X7R1H104MA; Product (none) -> CGA3E2X7R1H104M080AA
- J1101: Manufacturer (none) -> Neutrik; Mouser (none) -> 568-NE8FAH; Product (none) -> NE8FAH
- R1101: footprint Resistor_SMD:R_0603_1608Metric -> V2_Resistor_SMD:R_0603; symbol Device:R_Small -> V2_Device:R_0603_100R; Manufacturer (none) -> Vishay; Mouser (none) -> 71-CRCW0603100RFKEAH; Product (none) -> CRCW0603100RFKEAHP; Rating (none) -> 330mW
- U1101: value THVD24x2 -> THVD2442; symbol V2_Interface_RS485:THVD24x2 -> V2_Interface_RS485:THVD2442; Manufacturer (none) -> Texas Instruments; Mouser (none) -> 595-THVD2442DRCR; Product (none) -> THVD2442DRCR
Changed lines of the file:
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@@
 	)
 	(symbol
-		(lib_id "power:GND")
+		(lib_id "V2_power:GND")
 		(at 168.91 74.93 0)
 		(unit 1)
@@
 	)
 	(symbol
-		(lib_id "V2_Interface_RS485:THVD24x2")
+		(lib_id "V2_Interface_RS485:THVD2442")
 		(at 148.59 92.71 0)
 		(unit 1)
@@
 			)
 		)
-		(property "Value" "THVD24x2"
+		(property "Value" "THVD2442"
 			(at 150.7333 77.47 0)
 			(effects
@@
 		(property "Description" ""
 			(at 148.59 92.71 0)
+			(effects
+				(font
+					(size 1.27 1.27)
+				)
+				(hide yes)
+			)
+		)
+		(property "Mouser" "595-THVD2442DRCR"
+			(at 148.59 128.27 0)
+			(effects
+				(font
+					(size 1.27 1.27)
+				)
+				(hide yes)
+			)
+		)
+		(property "Product" "THVD2442DRCR "
+			(at 148.59 125.73 0)
+			(effects
+				(font
+					(size 1.27 1.27)
+				)
+				(hide yes)
+			)
+		)
+		(property "Manufacturer" "Texas Instruments"
+			(at 148.59 123.19 0)
 			(effects
 				(font
@@
 	)
 	(symbol
-		(lib_id "Device:R_Small")
+		(lib_id "V2_Device:R_0603_100R")
 		(at 161.29 87.63 0)
 		(unit 1)
@@
 		)
 		(property "Value" "100R"
-			(at 166.37 88.9 0)
-			(effects
-				(font
-					(size 1.27 1.27)
-				)
-			)
-		)
-		(property "Footprint" "Resistor_SMD:R_0603_1608Metric"
+			(at 165.1 88.9 0)
+			(effects
+				(font
+					(size 1.27 1.27)
+				)
+			)
+		)
+		(property "Footprint" "V2_Resistor_SMD:R_0603"
+			(at 161.29 103.378 0)
+			(effects
+				(font
+					(size 1.27 1.27)
+				)
+				(hide yes)
+			)
+		)
+		(property "Datasheet" ""
 			(at 161.29 87.63 0)
 			(effects
@@
 			)
 		)
-		(property "Datasheet" "~"
-			(at 161.29 87.63 0)
-			(effects
-				(font
-					(size 1.27 1.27)
-				)
-				(hide yes)
-			)
-		)
 		(property "Description" "Resistor, small symbol"
-			(at 161.29 87.63 0)
+			(at 161.29 102.87 0)
+			(effects
+				(font
+					(size 1.27 1.27)
+				)
+				(hide yes)
+			)
+		)
+		(property "Mouser" "71-CRCW0603100RFKEAH"
+			(at 161.29 113.03 0)
+			(effects
+				(font
+					(size 1.27 1.27)
+				)
+				(hide yes)
+			)
+		)
+		(property "Rating" "330mW"
+			(at 161.29 110.49 0)
+			(effects
+				(font
+					(size 1.27 1.27)
+				)
+				(hide yes)
+			)
+		)
+		(property "Manufacturer" "Vishay"
+			(at 161.29 105.41 0)
+			(effects
+				(font
+					(size 1.27 1.27)
+				)
+				(hide yes)
+			)
+		)
+		(property "Product" "CRCW0603100RFKEAHP"
+			(at 161.29 107.95 0)
 			(effects
 				(font
@@
 			)
 		)
-		(property "Sim.Enable" "0"
-			(at 148.59 137.16 0)
+		(property "Mouser" "568-NE8FAH"
+			(at 148.59 170.18 0)
+			(effects
+				(font
+					(size 1.27 1.27)
+				)
+				(hide yes)
+			)
+		)
+		(property "Manufacturer" "Neutrik"
+			(at 148.59 165.1 0)
+			(effects
+				(font
+					(size 1.27 1.27)
+				)
+				(hide yes)
+			)
+		)
+		(property "Product" "NE8FAH"
+			(at 148.59 167.64 0)
 			(effects
 				(font
@@
 	)
 	(symbol
-		(lib_id "power:GND")
+		(lib_id "V2_power:GND")
 		(at 148.59 107.95 0)
 		(unit 1)
@@
 	)
 	(symbol
-		(lib_id "power:+3V3")
+		(lib_id "V2_power:+3V3")
 		(at 148.59 69.85 0)
 		(unit 1)
@@
 	)
 	(symbol
-		(lib_id "Device:C_Small")
+		(lib_id "V2_Device:C_0603_0u1")
 		(at 168.91 72.39 0)
 		(unit 1)
@@
 		)
 		(property "Value" "0u1"
-			(at 173.99 73.6662 0)
-			(effects
-				(font
-					(size 1.27 1.27)
-				)
-			)
-		)
-		(property "Footprint" "Capacitor_SMD:C_0603_1608Metric"
+			(at 170.688 74.422 0)
+			(effects
+				(font
+					(size 1.27 1.27)
+				)
+				(justify left)
+			)
+		)
+		(property "Footprint" "V2_Capacitor_SMD:C_0603"
+			(at 168.91 89.408 0)
+			(effects
+				(font
+					(size 1.27 1.27)
+				)
+				(hide yes)
+			)
+		)
+		(property "Datasheet" ""
 			(at 168.91 72.39 0)
 			(effects
@@
 			)
 		)
-		(property "Datasheet" "~"
-			(at 168.91 72.39 0)
-			(effects
-				(font
-					(size 1.27 1.27)
-				)
-				(hide yes)
-			)
-		)
 		(property "Description" "Unpolarized capacitor, small symbol"
-			(at 168.91 72.39 0)
+			(at 168.91 85.09 0)
+			(effects
+				(font
+					(size 1.27 1.27)
+				)
+				(hide yes)
+			)
+		)
+		(property "Mouser" "810-CGA3E2X7R1H104MA"
+			(at 168.91 92.71 0)
+			(effects
+				(font
+					(size 1.27 1.27)
+				)
+				(hide yes)
+			)
+		)
+		(property "Manufacturer" "TDK"
+			(at 168.91 87.63 0)
+			(effects
+				(font
+					(size 1.27 1.27)
+				)
+				(hide yes)
+			)
+		)
+		(property "Product" "CGA3E2X7R1H104M080AA"
+			(at 168.91 90.17 0)
 			(effects
 				(font
@@
 	)
 	(symbol
-		(lib_id "power:GND")
+		(lib_id "V2_power:GND")
 		(at 138.43 127 270)
 		(mirror x)

Commit message: Replace Order_Number
Parts:
- C1101: Rating (none) -> 50V
Changed lines of the file:
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@@
 			)
 		)
-		(property "Description" "Power symbol creates a global label with name \"GND\" , ground"
+		(property "Description" ""
 			(at 168.91 74.93 0)
 			(effects
@@
 			)
 		)
-		(property "Description" "Power symbol creates a global label with name \"GND\" , ground"
+		(property "Description" ""
 			(at 148.59 107.95 0)
 			(effects
@@
 			)
 		)
-		(property "Description" "Power symbol creates a global label with name \"+3V3\""
+		(property "Description" ""
 			(at 148.59 69.85 0)
 			(effects
@@
 		(property "Product" "CGA3E2X7R1H104M080AA"
 			(at 168.91 90.17 0)
+			(effects
+				(font
+					(size 1.27 1.27)
+				)
+				(hide yes)
+			)
+		)
+		(property "Rating" "50V"
+			(at 168.91 95.25 0)
 			(effects
 				(font
@@
 			)
 		)
-		(property "Description" "Power symbol creates a global label with name \"GND\" , ground"
+		(property "Description" ""
 			(at 138.43 127 0)
 			(effects

Commit message: Update Library
Parts:
- C1101: symbol V2_Device:C_0603_0u1 -> V2_Capacitor:0603_0u1
- R1101: symbol V2_Device:R_0603_100R -> V2_Resistor:0603_100R
Changed lines of the file:
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@@
 		(on_board yes)
 		(dnp no)
-		(property "Reference" "#PWR01102"
+		(property "Reference" "#PWR1102"
 			(at 168.91 81.28 0)
 			(effects
@@
 			(project "sax"
 				(path "/6c8448b4-b04d-47e1-934e-e40cbe27a7be/be5efeaa-f0dd-4882-b2f8-53c61e0a33bd"
-					(reference "#PWR01102")
+					(reference "#PWR1102")
 					(unit 1)
 				)
@@
 	)
 	(symbol
-		(lib_id "V2_Device:R_0603_100R")
+		(lib_id "V2_Resistor:0603_100R")
 		(at 161.29 87.63 0)
 		(unit 1)
@@
 		(on_board yes)
 		(dnp no)
-		(property "Reference" "#PWR01103"
+		(property "Reference" "#PWR1103"
 			(at 148.59 114.3 0)
 			(effects
@@
 			(project "sax"
 				(path "/6c8448b4-b04d-47e1-934e-e40cbe27a7be/be5efeaa-f0dd-4882-b2f8-53c61e0a33bd"
-					(reference "#PWR01103")
+					(reference "#PWR1103")
 					(unit 1)
 				)
@@
 		(on_board yes)
 		(dnp no)
-		(property "Reference" "#PWR01101"
+		(property "Reference" "#PWR1101"
 			(at 148.59 73.66 0)
 			(effects
@@
 			(project "sax"
 				(path "/6c8448b4-b04d-47e1-934e-e40cbe27a7be/be5efeaa-f0dd-4882-b2f8-53c61e0a33bd"
-					(reference "#PWR01101")
+					(reference "#PWR1101")
 					(unit 1)
 				)
@@
 	)
 	(symbol
-		(lib_id "V2_Device:C_0603_0u1")
+		(lib_id "V2_Capacitor:0603_0u1")
 		(at 168.91 72.39 0)
 		(unit 1)
@@
 		(on_board yes)
 		(dnp no)
-		(property "Reference" "#PWR01104"
+		(property "Reference" "#PWR1104"
 			(at 132.08 127 0)
 			(effects
@@
 			(project "sax"
 				(path "/6c8448b4-b04d-47e1-934e-e40cbe27a7be/be5efeaa-f0dd-4882-b2f8-53c61e0a33bd"
-					(reference "#PWR01104")
-					(unit 1)
-				)
+					(reference "#PWR1104")
+					(unit 1)
+				)

Commit message: KiCad 10
Other:
- company: Plug -> Versio Duo

Commit message: Replace step-down
Other:
- title: V2 Link -> V2 sax
Changed lines of the file:
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@@
 	(paper "A4")
 	(title_block
-		(title "V2 Link")
-		(date "2026-03-21")
-		(rev "2026-02-10")
+		(title "V2 sax")
+		(date "2026-03-31")
+		(rev "2026-03-31")
 		(company "Versio Duo")
 	)
