File: hardware/sax/LinkPlug.kicad_sch (KiCad schematic)
At the start: 4 parts, among them J1101 NE8FAH, U1101 THVD2442

Commit message: Good Bye Imperial
Parts:
- C1101: footprint V2_Capacitor_SMD:C_0603 -> V2_Capacitor_SMD:C_1608; symbol V2_Capacitor:0603_0u1 -> V2_Capacitor:1608_0u1
- R1101: footprint V2_Resistor_SMD:R_0603 -> V2_Resistor_SMD:R_1608; symbol V2_Resistor:0603_100R -> V2_Resistor:1608_100R
Changed lines of the file:
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@@
 	)
 	(symbol
-		(lib_id "V2_Resistor:0603_100R")
+		(lib_id "V2_Resistor:1608_100R")
 		(at 161.29 87.63 0)
 		(unit 1)
@@
 			)
 		)
-		(property "Footprint" "V2_Resistor_SMD:R_0603"
+		(property "Footprint" "V2_Resistor_SMD:R_1608"
 			(at 161.29 103.378 0)
 			(hide yes)
@@
 	)
 	(symbol
-		(lib_id "V2_Capacitor:0603_0u1")
+		(lib_id "V2_Capacitor:1608_0u1")
 		(at 168.91 72.39 0)
 		(unit 1)
@@
 			)
 		)
-		(property "Footprint" "V2_Capacitor_SMD:C_0603"
+		(property "Footprint" "V2_Capacitor_SMD:C_1608"
 			(at 168.91 89.408 0)
 			(hide yes)

Commit message: Refresh
Parts:
- renumbered C1101 to C201, J1101 to J201, R1101 to R201, U1101 to U201
Changed lines of the file:
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@@
 	(title_block
 		(title "V2 sax")
-		(date "2026-04-23")
+		(date "2026-06-11")
 		(rev "2026-03-31")
 		(company "Versio Duo")
@@
 		(in_pos_files yes)
 		(dnp no)
-		(property "Reference" "#PWR01104"
+		(property "Reference" "#PWR0204"
 			(at 168.91 81.28 0)
 			(hide yes)
@@
 			(project "sax"
 				(path "/6c8448b4-b04d-47e1-934e-e40cbe27a7be/be5efeaa-f0dd-4882-b2f8-53c61e0a33bd"
-					(reference "#PWR01104")
+					(reference "#PWR0204")
 					(unit 1)
 				)
@@
 		(dnp no)
 		(fields_autoplaced yes)
-		(property "Reference" "U1101"
+		(property "Reference" "U201"
 			(at 150.7333 74.93 0)
 			(show_name no)
@@
 			(project "sax"
 				(path "/6c8448b4-b04d-47e1-934e-e40cbe27a7be/be5efeaa-f0dd-4882-b2f8-53c61e0a33bd"
-					(reference "U1101")
+					(reference "U201")
 					(unit 1)
 				)
@@
 		(in_pos_files yes)
 		(dnp no)
-		(property "Reference" "R1101"
+		(property "Reference" "R201"
 			(at 166.37 86.36 0)
 			(show_name no)
@@
 			(project "sax"
 				(path "/6c8448b4-b04d-47e1-934e-e40cbe27a7be/be5efeaa-f0dd-4882-b2f8-53c61e0a33bd"
-					(reference "R1101")
+					(reference "R201")
 					(unit 1)
 				)
@@
 		(dnp no)
 		(fields_autoplaced yes)
-		(property "Reference" "J1101"
+		(property "Reference" "J201"
 			(at 157.48 134.6199 0)
 			(show_name no)
@@
 			(project "sax"
 				(path "/6c8448b4-b04d-47e1-934e-e40cbe27a7be/be5efeaa-f0dd-4882-b2f8-53c61e0a33bd"
-					(reference "J1101")
+					(reference "J201")
 					(unit 1)
 				)
@@
 		(in_pos_files yes)
 		(dnp no)
-		(property "Reference" "#PWR01103"
+		(property "Reference" "#PWR0203"
 			(at 148.59 114.3 0)
 			(hide yes)
@@
 			(project "sax"
 				(path "/6c8448b4-b04d-47e1-934e-e40cbe27a7be/be5efeaa-f0dd-4882-b2f8-53c61e0a33bd"
-					(reference "#PWR01103")
+					(reference "#PWR0203")
 					(unit 1)
 				)
@@
 		(in_pos_files yes)
 		(dnp no)
-		(property "Reference" "#PWR01102"
+		(property "Reference" "#PWR0202"
 			(at 148.59 73.66 0)
 			(hide yes)
@@
 			(project "sax"
 				(path "/6c8448b4-b04d-47e1-934e-e40cbe27a7be/be5efeaa-f0dd-4882-b2f8-53c61e0a33bd"
-					(reference "#PWR01102")
+					(reference "#PWR0202")
 					(unit 1)
 				)
@@
 		(in_pos_files yes)
 		(dnp no)
-		(property "Reference" "C1101"
+		(property "Reference" "C201"
 			(at 171.45 71.1262 0)
 			(show_name no)
@@
 			(project "sax"
 				(path "/6c8448b4-b04d-47e1-934e-e40cbe27a7be/be5efeaa-f0dd-4882-b2f8-53c61e0a33bd"
-					(reference "C1101")
+					(reference "C201")
 					(unit 1)
 				)
@@
 		(in_pos_files yes)
 		(dnp no)
-		(property "Reference" "#PWR01101"
+		(property "Reference" "#PWR0201"
 			(at 132.08 127 0)
 			(hide yes)
@@
 			(project "sax"
 				(path "/6c8448b4-b04d-47e1-934e-e40cbe27a7be/be5efeaa-f0dd-4882-b2f8-53c61e0a33bd"
-					(reference "#PWR01101")
+					(reference "#PWR0201")
 					(unit 1)
 				)
