File: hardware/sax/OrientationSensor.kicad_sch (KiCad schematic)
At the start: 10 parts, among them U1401 BMM150, U1402 BHI160

Commit message: Update
Parts:
- renumbered C1401 to C1402, C1406 to C1403, C1404 to C1406, D1403 to D1402, R1406 to R1405, R1407 to R1406, U1402 to U1401, U1401 to U1402
Changed lines of the file:
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@@
 	(title_block
 		(title "V2 sax")
-		(date "2026-04-10")
+		(date "2026-04-23")
 		(rev "2026-03-31")
 		(company "Versio Duo")
@@
 		(in_pos_files yes)
 		(dnp no)
-		(property "Reference" "C1401"
+		(property "Reference" "C1402"
 			(at 131.445 78.74 0)
 			(show_name no)
@@
 			(project "sax"
 				(path "/6c8448b4-b04d-47e1-934e-e40cbe27a7be/f7096e67-1c66-4074-b306-32741be5ff9b"
-					(reference "C1401")
+					(reference "C1402")
 					(unit 1)
 				)
@@
 		(in_pos_files yes)
 		(dnp no)
-		(property "Reference" "#PWR1403"
+		(property "Reference" "#PWR01401"
 			(at 93.98 87.63 0)
 			(hide yes)
@@
 			(project "sax"
 				(path "/6c8448b4-b04d-47e1-934e-e40cbe27a7be/f7096e67-1c66-4074-b306-32741be5ff9b"
-					(reference "#PWR1403")
+					(reference "#PWR01401")
 					(unit 1)
 				)
@@
 		(in_pos_files yes)
 		(dnp no)
-		(property "Reference" "R1406"
+		(property "Reference" "R1405"
 			(at 139.7 95.25 0)
 			(show_name no)
@@
 			(project "sax"
 				(path "/6c8448b4-b04d-47e1-934e-e40cbe27a7be/f7096e67-1c66-4074-b306-32741be5ff9b"
-					(reference "R1406")
+					(reference "R1405")
 					(unit 1)
 				)
@@
 		(in_pos_files yes)
 		(dnp no)
-		(property "Reference" "#PWR1401"
+		(property "Reference" "#PWR01404"
 			(at 124.46 81.28 0)
 			(hide yes)
@@
 			(project "sax"
 				(path "/6c8448b4-b04d-47e1-934e-e40cbe27a7be/f7096e67-1c66-4074-b306-32741be5ff9b"
-					(reference "#PWR1401")
+					(reference "#PWR01404")
 					(unit 1)
 				)
@@
 		(in_pos_files yes)
 		(dnp no)
-		(property "Reference" "#PWR1428"
+		(property "Reference" "#PWR01417"
 			(at 166.37 146.05 0)
 			(hide yes)
@@
 			(project "sax"
 				(path "/6c8448b4-b04d-47e1-934e-e40cbe27a7be/f7096e67-1c66-4074-b306-32741be5ff9b"
-					(reference "#PWR1428")
+					(reference "#PWR01417")
 					(unit 1)
 				)
@@
 		(in_pos_files yes)
 		(dnp no)
-		(property "Reference" "#PWR1415"
+		(property "Reference" "#PWR01409"
 			(at 138.43 97.79 0)
 			(hide yes)
@@
 			(project "sax"
 				(path "/6c8448b4-b04d-47e1-934e-e40cbe27a7be/f7096e67-1c66-4074-b306-32741be5ff9b"
-					(reference "#PWR1415")
+					(reference "#PWR01409")
 					(unit 1)
 				)
@@
 		(in_pos_files yes)
 		(dnp no)
-		(property "Reference" "#PWR1420"
+		(property "Reference" "#PWR01426"
 			(at 214.63 106.68 0)
 			(hide yes)
@@
 			(project "sax"
 				(path "/6c8448b4-b04d-47e1-934e-e40cbe27a7be/f7096e67-1c66-4074-b306-32741be5ff9b"
-					(reference "#PWR1420")
+					(reference "#PWR01426")
 					(unit 1)
 				)
@@
 		(in_pos_files yes)
 		(dnp no)
-		(property "Reference" "C1404"
+		(property "Reference" "C1406"
 			(at 215.9 92.71 0)
 			(show_name no)
@@
 			(project "sax"
 				(path "/6c8448b4-b04d-47e1-934e-e40cbe27a7be/f7096e67-1c66-4074-b306-32741be5ff9b"
-					(reference "C1404")
+					(reference "C1406")
 					(unit 1)
 				)
@@
 		(in_pos_files yes)
 		(dnp no)
-		(property "Reference" "#PWR1410"
+		(property "Reference" "#PWR01428"
 			(at 213.36 101.6 0)
 			(hide yes)
@@
 			(project "sax"
 				(path "/6c8448b4-b04d-47e1-934e-e40cbe27a7be/f7096e67-1c66-4074-b306-32741be5ff9b"
-					(reference "#PWR1410")
+					(reference "#PWR01428")
 					(unit 1)
 				)
@@
 		(in_pos_files yes)
 		(dnp no)
-		(property "Reference" "#PWR1402"
+		(property "Reference" "#PWR01408"
 			(at 129.54 88.9 0)
 			(hide yes)
@@
 			(project "sax"
 				(path "/6c8448b4-b04d-47e1-934e-e40cbe27a7be/f7096e67-1c66-4074-b306-32741be5ff9b"
-					(reference "#PWR1402")
+					(reference "#PWR01408")
 					(unit 1)
 				)
@@
 		(in_pos_files yes)
 		(dnp no)
-		(property "Reference" "#PWR1408"
+		(property "Reference" "#PWR01411"
 			(at 149.86 97.79 0)
 			(hide yes)
@@
 			(project "sax"
 				(path "/6c8448b4-b04d-47e1-934e-e40cbe27a7be/f7096e67-1c66-4074-b306-32741be5ff9b"
-					(reference "#PWR1408")
+					(reference "#PWR01411")
 					(unit 1)
 				)
@@
 		(in_pos_files yes)
 		(dnp no)
-		(property "Reference" "D1403"
+		(property "Reference" "D1402"
 			(at 149.606 134.62 0)
 			(show_name no)
@@
 			(project "sax"
 				(path "/6c8448b4-b04d-47e1-934e-e40cbe27a7be/f7096e67-1c66-4074-b306-32741be5ff9b"
-					(reference "D1403")
+					(reference "D1402")
 					(unit 1)
 				)
@@
 		(in_pos_files yes)
 		(dnp no)
-		(property "Reference" "U1401"
+		(property "Reference" "U1402"
 			(at 194.31 83.82 0)
 			(show_name no)
@@
 			(project "sax"
 				(path "/6c8448b4-b04d-47e1-934e-e40cbe27a7be/f7096e67-1c66-4074-b306-32741be5ff9b"
-					(reference "U1401")
+					(reference "U1402")
 					(unit 1)
 				)
@@
 		(in_pos_files yes)
 		(dnp no)
-		(property "Reference" "C1406"
+		(property "Reference" "C1403"
 			(at 132.715 92.075 90)
 			(show_name no)
@@
 			(project "sax"
 				(path "/6c8448b4-b04d-47e1-934e-e40cbe27a7be/f7096e67-1c66-4074-b306-32741be5ff9b"
-					(reference "C1406")
+					(reference "C1403")
 					(unit 1)
 				)
@@
 		(in_pos_files yes)
 		(dnp no)
-		(property "Reference" "#PWR1419"
+		(property "Reference" "#PWR01425"
 			(at 194.31 106.68 0)
 			(hide yes)
@@
 			(project "sax"
 				(path "/6c8448b4-b04d-47e1-934e-e40cbe27a7be/f7096e67-1c66-4074-b306-32741be5ff9b"
-					(reference "#PWR1419")
+					(reference "#PWR01425")
 					(unit 1)
 				)
@@
 		(in_pos_files yes)
 		(dnp no)
-		(property "Reference" "#PWR1417"
+		(property "Reference" "#PWR01424"
 			(at 184.15 99.06 0)
 			(hide yes)
@@
 			(project "sax"
 				(path "/6c8448b4-b04d-47e1-934e-e40cbe27a7be/f7096e67-1c66-4074-b306-32741be5ff9b"
-					(reference "#PWR1417")
+					(reference "#PWR01424")
 					(unit 1)
 				)
@@
 		(in_pos_files yes)
 		(dnp no)
-		(property "Reference" "#PWR1409"
+		(property "Reference" "#PWR01423"
 			(at 184.15 93.98 0)
 			(hide yes)
@@
 			(project "sax"
 				(path "/6c8448b4-b04d-47e1-934e-e40cbe27a7be/f7096e67-1c66-4074-b306-32741be5ff9b"
-					(reference "#PWR1409")
+					(reference "#PWR01423")
 					(unit 1)
 				)
@@
 		(in_pos_files yes)
 		(dnp no)
-		(property "Reference" "#PWR1406"
+		(property "Reference" "#PWR01427"
 			(at 213.36 95.25 0)
 			(hide yes)
@@
 			(project "sax"
 				(path "/6c8448b4-b04d-47e1-934e-e40cbe27a7be/f7096e67-1c66-4074-b306-32741be5ff9b"
-					(reference "#PWR1406")
+					(reference "#PWR01427")
 					(unit 1)
 				)
@@
 		(in_pos_files yes)
 		(dnp no)
-		(property "Reference" "#PWR1421"
+		(property "Reference" "#PWR01402"
 			(at 97.79 107.95 0)
 			(hide yes)
@@
 			(project "sax"
 				(path "/6c8448b4-b04d-47e1-934e-e40cbe27a7be/f7096e67-1c66-4074-b306-32741be5ff9b"
-					(reference "#PWR1421")
+					(reference "#PWR01402")
 					(unit 1)
 				)
@@
 		(in_pos_files yes)
 		(dnp no)
-		(property "Reference" "U1402"
+		(property "Reference" "U1401"
 			(at 109.982 85.344 0)
 			(show_name no)
@@
 			(project "sax"
 				(path "/6c8448b4-b04d-47e1-934e-e40cbe27a7be/f7096e67-1c66-4074-b306-32741be5ff9b"
-					(reference "U1402")
+					(reference "U1401")
 					(unit 1)
 				)
@@
 		(in_pos_files yes)
 		(dnp no)
-		(property "Reference" "R1407"
+		(property "Reference" "R1406"
 			(at 153.035 95.25 0)
 			(show_name no)
@@
 			(project "sax"
 				(path "/6c8448b4-b04d-47e1-934e-e40cbe27a7be/f7096e67-1c66-4074-b306-32741be5ff9b"
-					(reference "R1407")
+					(reference "R1406")
 					(unit 1)
 				)
@@
 		(in_pos_files yes)
 		(dnp no)
-		(property "Reference" "#PWR1427"
+		(property "Reference" "#PWR01416"
 			(at 156.21 140.97 0)
 			(hide yes)
@@
 			(project "sax"
 				(path "/6c8448b4-b04d-47e1-934e-e40cbe27a7be/f7096e67-1c66-4074-b306-32741be5ff9b"
-					(reference "#PWR1427")
+					(reference "#PWR01416")
 					(unit 1)
 				)
@@
 		(in_pos_files yes)
 		(dnp no)
-		(property "Reference" "#PWR1422"
+		(property "Reference" "#PWR01405"
 			(at 130.81 113.03 0)
 			(hide yes)
@@
 			(project "sax"
 				(path "/6c8448b4-b04d-47e1-934e-e40cbe27a7be/f7096e67-1c66-4074-b306-32741be5ff9b"
-					(reference "#PWR1422")
+					(reference "#PWR01405")
 					(unit 1)
 				)

Commit message: Good Bye Imperial
Parts:
- C1402: footprint V2_Capacitor_SMD:C_0603 -> V2_Capacitor_SMD:C_1608; symbol V2_Capacitor:0603_10u -> V2_Capacitor:1608_10u
- C1403: footprint V2_Capacitor_SMD:C_0603 -> V2_Capacitor_SMD:C_1608; symbol V2_Capacitor:0603_0u47 -> V2_Capacitor:1608_0u47
- C1406: footprint V2_Capacitor_SMD:C_0603 -> V2_Capacitor_SMD:C_1608; symbol V2_Capacitor:0603_0u1 -> V2_Capacitor:1608_0u1
- R1401, R1402, R1405, R1406: footprint V2_Resistor_SMD:R_0603 -> V2_Resistor_SMD:R_1608; symbol V2_Resistor:0603_2k7 -> V2_Resistor:1608_2k7
Changed lines of the file:
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@@
 	)
 	(symbol
-		(lib_id "V2_Capacitor:0603_10u")
+		(lib_id "V2_Capacitor:1608_10u")
 		(at 129.54 80.01 0)
 		(unit 1)
@@
 			)
 		)
-		(property "Footprint" "V2_Capacitor_SMD:C_0603"
+		(property "Footprint" "V2_Capacitor_SMD:C_1608"
 			(at 129.54 97.028 0)
 			(hide yes)
@@
 	)
 	(symbol
-		(lib_id "V2_Resistor:0603_2k7")
+		(lib_id "V2_Resistor:1608_2k7")
 		(at 95.25 86.36 0)
 		(unit 1)
@@
 			)
 		)
-		(property "Footprint" "V2_Resistor_SMD:R_0603"
+		(property "Footprint" "V2_Resistor_SMD:R_1608"
 			(at 95.25 102.108 0)
 			(hide yes)
@@
 	)
 	(symbol
-		(lib_id "V2_Resistor:0603_2k7")
+		(lib_id "V2_Resistor:1608_2k7")
 		(at 148.59 96.52 0)
 		(unit 1)
@@
 			)
 		)
-		(property "Footprint" "V2_Resistor_SMD:R_0603"
+		(property "Footprint" "V2_Resistor_SMD:R_1608"
 			(at 148.59 112.268 0)
 			(hide yes)
@@
 	)
 	(symbol
-		(lib_id "V2_Resistor:0603_2k7")
+		(lib_id "V2_Resistor:1608_2k7")
 		(at 92.71 86.36 0)
 		(unit 1)
@@
 			)
 		)
-		(property "Footprint" "V2_Resistor_SMD:R_0603"
+		(property "Footprint" "V2_Resistor_SMD:R_1608"
 			(at 92.71 102.108 0)
 			(hide yes)
@@
 	)
 	(symbol
-		(lib_id "V2_Capacitor:0603_0u1")
+		(lib_id "V2_Capacitor:1608_0u1")
 		(at 213.36 93.98 0)
 		(unit 1)
@@
 			)
 		)
-		(property "Footprint" "V2_Capacitor_SMD:C_0603"
+		(property "Footprint" "V2_Capacitor_SMD:C_1608"
 			(at 213.36 110.998 0)
 			(hide yes)
@@
 	)
 	(symbol
-		(lib_id "V2_Capacitor:0603_0u47")
+		(lib_id "V2_Capacitor:1608_0u47")
 		(at 129.54 97.79 90)
 		(unit 1)
@@
 			)
 		)
-		(property "Footprint" "V2_Capacitor_SMD:C_0603"
+		(property "Footprint" "V2_Capacitor_SMD:C_1608"
 			(at 146.558 97.79 0)
 			(hide yes)
@@
 	)
 	(symbol
-		(lib_id "V2_Resistor:0603_2k7")
+		(lib_id "V2_Resistor:1608_2k7")
 		(at 151.13 96.52 0)
 		(unit 1)
@@
 			)
 		)
-		(property "Footprint" "V2_Resistor_SMD:R_0603"
+		(property "Footprint" "V2_Resistor_SMD:R_1608"
 			(at 151.13 112.268 0)
 			(hide yes)

Commit message: Refresh
Parts:
- renumbered C1402 to C1301, C1403 to C1302, C1406 to C1303, D1402 to D1301, R1401 to R1301, R1402 to R1302, R1405 to R1303, R1406 to R1304, U1401 to U1301, U1402 to U1302
Changed lines of the file:
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@@
 	(title_block
 		(title "V2 sax")
-		(date "2026-04-23")
+		(date "2026-06-11")
 		(rev "2026-03-31")
 		(company "Versio Duo")
@@
 		(in_pos_files yes)
 		(dnp no)
-		(property "Reference" "C1402"
+		(property "Reference" "C1301"
 			(at 131.445 78.74 0)
 			(show_name no)
@@
 			(project "sax"
 				(path "/6c8448b4-b04d-47e1-934e-e40cbe27a7be/f7096e67-1c66-4074-b306-32741be5ff9b"
-					(reference "C1402")
+					(reference "C1301")
 					(unit 1)
 				)
@@
 		(in_pos_files yes)
 		(dnp no)
-		(property "Reference" "R1402"
+		(property "Reference" "R1302"
 			(at 97.0702 85.1591 0)
 			(show_name no)
@@
 			(project "sax"
 				(path "/6c8448b4-b04d-47e1-934e-e40cbe27a7be/f7096e67-1c66-4074-b306-32741be5ff9b"
-					(reference "R1402")
+					(reference "R1302")
 					(unit 1)
 				)
@@
 		(in_pos_files yes)
 		(dnp no)
-		(property "Reference" "#PWR01401"
+		(property "Reference" "#PWR01301"
 			(at 93.98 87.63 0)
 			(hide yes)
@@
 			(project "sax"
 				(path "/6c8448b4-b04d-47e1-934e-e40cbe27a7be/f7096e67-1c66-4074-b306-32741be5ff9b"
-					(reference "#PWR01401")
+					(reference "#PWR01301")
 					(unit 1)
 				)
@@
 		(in_pos_files yes)
 		(dnp no)
-		(property "Reference" "R1405"
+		(property "Reference" "R1303"
 			(at 139.7 95.25 0)
 			(show_name no)
@@
 			(project "sax"
 				(path "/6c8448b4-b04d-47e1-934e-e40cbe27a7be/f7096e67-1c66-4074-b306-32741be5ff9b"
-					(reference "R1405")
+					(reference "R1303")
 					(unit 1)
 				)
@@
 		(in_pos_files yes)
 		(dnp no)
-		(property "Reference" "R1401"
+		(property "Reference" "R1301"
 			(at 83.82 84.836 0)
 			(show_name no)
@@
 			(project "sax"
 				(path "/6c8448b4-b04d-47e1-934e-e40cbe27a7be/f7096e67-1c66-4074-b306-32741be5ff9b"
-					(reference "R1401")
+					(reference "R1301")
 					(unit 1)
 				)
@@
 		(in_pos_files yes)
 		(dnp no)
-		(property "Reference" "#PWR01404"
+		(property "Reference" "#PWR01303"
 			(at 124.46 81.28 0)
 			(hide yes)
@@
 			(project "sax"
 				(path "/6c8448b4-b04d-47e1-934e-e40cbe27a7be/f7096e67-1c66-4074-b306-32741be5ff9b"
-					(reference "#PWR01404")
+					(reference "#PWR01303")
 					(unit 1)
 				)
@@
 		(in_pos_files yes)
 		(dnp no)
-		(property "Reference" "#PWR01417"
+		(property "Reference" "#PWR01309"
 			(at 166.37 146.05 0)
 			(hide yes)
@@
 			(project "sax"
 				(path "/6c8448b4-b04d-47e1-934e-e40cbe27a7be/f7096e67-1c66-4074-b306-32741be5ff9b"
-					(reference "#PWR01417")
+					(reference "#PWR01309")
 					(unit 1)
 				)
@@
 		(in_pos_files yes)
 		(dnp no)
-		(property "Reference" "#PWR01409"
+		(property "Reference" "#PWR01306"
 			(at 138.43 97.79 0)
 			(hide yes)
@@
 			(project "sax"
 				(path "/6c8448b4-b04d-47e1-934e-e40cbe27a7be/f7096e67-1c66-4074-b306-32741be5ff9b"
-					(reference "#PWR01409")
+					(reference "#PWR01306")
 					(unit 1)
 				)
@@
 		(in_pos_files yes)
 		(dnp no)
-		(property "Reference" "#PWR01426"
+		(property "Reference" "#PWR01313"
 			(at 214.63 106.68 0)
 			(hide yes)
@@
 			(project "sax"
 				(path "/6c8448b4-b04d-47e1-934e-e40cbe27a7be/f7096e67-1c66-4074-b306-32741be5ff9b"
-					(reference "#PWR01426")
+					(reference "#PWR01313")
 					(unit 1)
 				)
@@
 		(in_pos_files yes)
 		(dnp no)
-		(property "Reference" "C1406"
+		(property "Reference" "C1303"
 			(at 215.9 92.71 0)
 			(show_name no)
@@
 			(project "sax"
 				(path "/6c8448b4-b04d-47e1-934e-e40cbe27a7be/f7096e67-1c66-4074-b306-32741be5ff9b"
-					(reference "C1406")
+					(reference "C1303")
 					(unit 1)
 				)
@@
 		(in_pos_files yes)
 		(dnp no)
-		(property "Reference" "#PWR01428"
+		(property "Reference" "#PWR01315"
 			(at 213.36 101.6 0)
 			(hide yes)
@@
 			(project "sax"
 				(path "/6c8448b4-b04d-47e1-934e-e40cbe27a7be/f7096e67-1c66-4074-b306-32741be5ff9b"
-					(reference "#PWR01428")
+					(reference "#PWR01315")
 					(unit 1)
 				)
@@
 		(in_pos_files yes)
 		(dnp no)
-		(property "Reference" "#PWR01408"
+		(property "Reference" "#PWR01305"
 			(at 129.54 88.9 0)
 			(hide yes)
@@
 			(project "sax"
 				(path "/6c8448b4-b04d-47e1-934e-e40cbe27a7be/f7096e67-1c66-4074-b306-32741be5ff9b"
-					(reference "#PWR01408")
+					(reference "#PWR01305")
 					(unit 1)
 				)
@@
 		(in_pos_files yes)
 		(dnp no)
-		(property "Reference" "#PWR01411"
+		(property "Reference" "#PWR01307"
 			(at 149.86 97.79 0)
 			(hide yes)
@@
 			(project "sax"
 				(path "/6c8448b4-b04d-47e1-934e-e40cbe27a7be/f7096e67-1c66-4074-b306-32741be5ff9b"
-					(reference "#PWR01411")
+					(reference "#PWR01307")
 					(unit 1)
 				)
@@
 		(in_pos_files yes)
 		(dnp no)
-		(property "Reference" "D1402"
+		(property "Reference" "D1301"
 			(at 149.606 134.62 0)
 			(show_name no)
@@
 			(project "sax"
 				(path "/6c8448b4-b04d-47e1-934e-e40cbe27a7be/f7096e67-1c66-4074-b306-32741be5ff9b"
-					(reference "D1402")
+					(reference "D1301")
 					(unit 1)
 				)
@@
 		(in_pos_files yes)
 		(dnp no)
-		(property "Reference" "U1402"
+		(property "Reference" "U1302"
 			(at 194.31 83.82 0)
 			(show_name no)
@@
 			(project "sax"
 				(path "/6c8448b4-b04d-47e1-934e-e40cbe27a7be/f7096e67-1c66-4074-b306-32741be5ff9b"
-					(reference "U1402")
+					(reference "U1302")
 					(unit 1)
 				)
@@
 		(in_pos_files yes)
 		(dnp no)
-		(property "Reference" "C1403"
+		(property "Reference" "C1302"
 			(at 132.715 92.075 90)
 			(show_name no)
@@
 			(project "sax"
 				(path "/6c8448b4-b04d-47e1-934e-e40cbe27a7be/f7096e67-1c66-4074-b306-32741be5ff9b"
-					(reference "C1403")
+					(reference "C1302")
 					(unit 1)
 				)
@@
 		(in_pos_files yes)
 		(dnp no)
-		(property "Reference" "#PWR01425"
+		(property "Reference" "#PWR01312"
 			(at 194.31 106.68 0)
 			(hide yes)
@@
 			(project "sax"
 				(path "/6c8448b4-b04d-47e1-934e-e40cbe27a7be/f7096e67-1c66-4074-b306-32741be5ff9b"
-					(reference "#PWR01425")
+					(reference "#PWR01312")
 					(unit 1)
 				)
@@
 		(in_pos_files yes)
 		(dnp no)
-		(property "Reference" "#PWR01424"
+		(property "Reference" "#PWR01311"
 			(at 184.15 99.06 0)
 			(hide yes)
@@
 			(project "sax"
 				(path "/6c8448b4-b04d-47e1-934e-e40cbe27a7be/f7096e67-1c66-4074-b306-32741be5ff9b"
-					(reference "#PWR01424")
+					(reference "#PWR01311")
 					(unit 1)
 				)
@@
 		(in_pos_files yes)
 		(dnp no)
-		(property "Reference" "#PWR01423"
+		(property "Reference" "#PWR01310"
 			(at 184.15 93.98 0)
 			(hide yes)
@@
 			(project "sax"
 				(path "/6c8448b4-b04d-47e1-934e-e40cbe27a7be/f7096e67-1c66-4074-b306-32741be5ff9b"
-					(reference "#PWR01423")
+					(reference "#PWR01310")
 					(unit 1)
 				)
@@
 		(in_pos_files yes)
 		(dnp no)
-		(property "Reference" "#PWR01427"
+		(property "Reference" "#PWR01314"
 			(at 213.36 95.25 0)
 			(hide yes)
@@
 			(project "sax"
 				(path "/6c8448b4-b04d-47e1-934e-e40cbe27a7be/f7096e67-1c66-4074-b306-32741be5ff9b"
-					(reference "#PWR01427")
+					(reference "#PWR01314")
 					(unit 1)
 				)
@@
 		(in_pos_files yes)
 		(dnp no)
-		(property "Reference" "#PWR01402"
+		(property "Reference" "#PWR01302"
 			(at 97.79 107.95 0)
 			(hide yes)
@@
 			(project "sax"
 				(path "/6c8448b4-b04d-47e1-934e-e40cbe27a7be/f7096e67-1c66-4074-b306-32741be5ff9b"
-					(reference "#PWR01402")
+					(reference "#PWR01302")
 					(unit 1)
 				)
@@
 		(in_pos_files yes)
 		(dnp no)
-		(property "Reference" "U1401"
+		(property "Reference" "U1301"
 			(at 109.982 85.344 0)
 			(show_name no)
@@
 			(project "sax"
 				(path "/6c8448b4-b04d-47e1-934e-e40cbe27a7be/f7096e67-1c66-4074-b306-32741be5ff9b"
-					(reference "U1401")
+					(reference "U1301")
 					(unit 1)
 				)
@@
 		(in_pos_files yes)
 		(dnp no)
-		(property "Reference" "R1406"
+		(property "Reference" "R1304"
 			(at 153.035 95.25 0)
 			(show_name no)
@@
 			(project "sax"
 				(path "/6c8448b4-b04d-47e1-934e-e40cbe27a7be/f7096e67-1c66-4074-b306-32741be5ff9b"
-					(reference "R1406")
+					(reference "R1304")
 					(unit 1)
 				)
@@
 		(in_pos_files yes)
 		(dnp no)
-		(property "Reference" "#PWR01416"
+		(property "Reference" "#PWR01308"
 			(at 156.21 140.97 0)
 			(hide yes)
@@
 			(project "sax"
 				(path "/6c8448b4-b04d-47e1-934e-e40cbe27a7be/f7096e67-1c66-4074-b306-32741be5ff9b"
-					(reference "#PWR01416")
+					(reference "#PWR01308")
 					(unit 1)
 				)
@@
 		(in_pos_files yes)
 		(dnp no)
-		(property "Reference" "#PWR01405"
+		(property "Reference" "#PWR01304"
 			(at 130.81 113.03 0)
 			(hide yes)
@@
 			(project "sax"
 				(path "/6c8448b4-b04d-47e1-934e-e40cbe27a7be/f7096e67-1c66-4074-b306-32741be5ff9b"
-					(reference "#PWR01405")
+					(reference "#PWR01304")
 					(unit 1)
 				)
