File: hardware/sax/PressureSensor.kicad_sch (KiCad schematic)
At the start: 5 parts, among them IC1401 MP3V5004GP

Commit message: Update
Parts:
- renumbered C1402 to C1401, C1403 to C1404, D1402 to D1403, R1404 to R1407
Changed lines of the file:
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@@
 	(title_block
 		(title "V2 sax")
-		(date "2026-04-10")
+		(date "2026-04-23")
 		(rev "2026-03-31")
 		(company "Versio Duo")
@@
 		(in_pos_files yes)
 		(dnp no)
-		(property "Reference" "C1403"
+		(property "Reference" "C1404"
 			(at 168.148 93.98 0)
 			(show_name no)
@@
 			(project "sax"
 				(path "/6c8448b4-b04d-47e1-934e-e40cbe27a7be/6178bc16-76cb-41ae-a61c-619a3590ea5a"
-					(reference "C1403")
+					(reference "C1404")
 					(unit 1)
 				)
@@
 		(dnp no)
 		(fields_autoplaced yes)
-		(property "Reference" "#PWR1407"
+		(property "Reference" "#PWR01407"
 			(at 125.73 100.33 0)
 			(hide yes)
@@
 			(project "sax"
 				(path "/6c8448b4-b04d-47e1-934e-e40cbe27a7be/6178bc16-76cb-41ae-a61c-619a3590ea5a"
-					(reference "#PWR1407")
+					(reference "#PWR01407")
 					(unit 1)
 				)
@@
 		(in_pos_files yes)
 		(dnp no)
-		(property "Reference" "#PWR1405"
+		(property "Reference" "#PWR01406"
 			(at 125.73 92.71 0)
 			(hide yes)
@@
 			(project "sax"
 				(path "/6c8448b4-b04d-47e1-934e-e40cbe27a7be/6178bc16-76cb-41ae-a61c-619a3590ea5a"
-					(reference "#PWR1405")
+					(reference "#PWR01406")
 					(unit 1)
 				)
@@
 		(in_pos_files yes)
 		(dnp no)
-		(property "Reference" "#PWR1404"
+		(property "Reference" "#PWR01412"
 			(at 152.4 86.36 0)
 			(hide yes)
@@
 			(project "sax"
 				(path "/6c8448b4-b04d-47e1-934e-e40cbe27a7be/6178bc16-76cb-41ae-a61c-619a3590ea5a"
-					(reference "#PWR1404")
+					(reference "#PWR01412")
 					(unit 1)
 				)
@@
 		(dnp no)
 		(fields_autoplaced yes)
-		(property "Reference" "#PWR1413"
+		(property "Reference" "#PWR01421"
 			(at 177.8 102.87 0)
 			(hide yes)
@@
 			(project "sax"
 				(path "/6c8448b4-b04d-47e1-934e-e40cbe27a7be/6178bc16-76cb-41ae-a61c-619a3590ea5a"
-					(reference "#PWR1413")
+					(reference "#PWR01421")
 					(unit 1)
 				)
@@
 		(in_pos_files yes)
 		(dnp no)
-		(property "Reference" "C1402"
+		(property "Reference" "C1401"
 			(at 128.27 90.17 0)
 			(show_name no)
@@
 			(project "sax"
 				(path "/6c8448b4-b04d-47e1-934e-e40cbe27a7be/6178bc16-76cb-41ae-a61c-619a3590ea5a"
-					(reference "C1402")
+					(reference "C1401")
 					(unit 1)
 				)
@@
 		(dnp no)
 		(fields_autoplaced yes)
-		(property "Reference" "#PWR1412"
+		(property "Reference" "#PWR01420"
 			(at 165.1 102.87 0)
 			(hide yes)
@@
 			(project "sax"
 				(path "/6c8448b4-b04d-47e1-934e-e40cbe27a7be/6178bc16-76cb-41ae-a61c-619a3590ea5a"
-					(reference "#PWR1412")
+					(reference "#PWR01420")
 					(unit 1)
 				)
@@
 		(dnp no)
 		(fields_autoplaced yes)
-		(property "Reference" "#PWR1411"
+		(property "Reference" "#PWR01413"
 			(at 162.56 96.52 0)
 			(hide yes)
@@
 			(project "sax"
 				(path "/6c8448b4-b04d-47e1-934e-e40cbe27a7be/6178bc16-76cb-41ae-a61c-619a3590ea5a"
-					(reference "#PWR1411")
+					(reference "#PWR01413")
 					(unit 1)
 				)
@@
 		(in_pos_files yes)
 		(dnp no)
-		(property "Reference" "D1402"
+		(property "Reference" "D1403"
 			(at 150.876 120.65 0)
 			(show_name no)
@@
 			(project "sax"
 				(path "/6c8448b4-b04d-47e1-934e-e40cbe27a7be/6178bc16-76cb-41ae-a61c-619a3590ea5a"
-					(reference "D1402")
+					(reference "D1403")
 					(unit 1)
 				)
@@
 		(in_pos_files yes)
 		(dnp no)
-		(property "Reference" "#PWR1424"
+		(property "Reference" "#PWR01418"
 			(at 157.48 127 0)
 			(hide yes)
@@
 			(project "sax"
 				(path "/6c8448b4-b04d-47e1-934e-e40cbe27a7be/6178bc16-76cb-41ae-a61c-619a3590ea5a"
-					(reference "#PWR1424")
+					(reference "#PWR01418")
 					(unit 1)
 				)
@@
 		(in_pos_files yes)
 		(dnp no)
-		(property "Reference" "R1404"
+		(property "Reference" "R1407"
 			(at 185.42 93.9799 0)
 			(show_name no)
@@
 			(project "sax"
 				(path "/6c8448b4-b04d-47e1-934e-e40cbe27a7be/6178bc16-76cb-41ae-a61c-619a3590ea5a"
-					(reference "R1404")
+					(reference "R1407")
 					(unit 1)
 				)
@@
 		(in_pos_files yes)
 		(dnp no)
-		(property "Reference" "#PWR1426"
+		(property "Reference" "#PWR01419"
 			(at 167.64 132.08 0)
 			(hide yes)
@@
 			(project "sax"
 				(path "/6c8448b4-b04d-47e1-934e-e40cbe27a7be/6178bc16-76cb-41ae-a61c-619a3590ea5a"
-					(reference "#PWR1426")
+					(reference "#PWR01419")
 					(unit 1)
 				)

Commit message: Good Bye Imperial
Parts:
- C1401: footprint V2_Capacitor_SMD:C_0603 -> V2_Capacitor_SMD:C_1608; symbol V2_Capacitor:0603_0u1 -> V2_Capacitor:1608_0u1
- C1404: footprint V2_Capacitor_SMD:C_0603 -> V2_Capacitor_SMD:C_1608; symbol V2_Capacitor:0603_0u022 -> V2_Capacitor:1608_0u022
- R1407: footprint V2_Resistor_SMD:R_0603 -> V2_Resistor_SMD:R_1608; symbol V2_Resistor:0603_100k -> V2_Resistor:1608_100k
Changed lines of the file:
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@@
 	)
 	(symbol
-		(lib_id "V2_Capacitor:0603_0u022")
+		(lib_id "V2_Capacitor:1608_0u022")
 		(at 165.1 93.98 0)
 		(unit 1)
@@
 			)
 		)
-		(property "Footprint" "V2_Capacitor_SMD:C_0603"
+		(property "Footprint" "V2_Capacitor_SMD:C_1608"
 			(at 165.1 110.998 0)
 			(hide yes)
@@
 	)
 	(symbol
-		(lib_id "V2_Capacitor:0603_0u1")
+		(lib_id "V2_Capacitor:1608_0u1")
 		(at 125.73 91.44 0)
 		(unit 1)
@@
 			)
 		)
-		(property "Footprint" "V2_Capacitor_SMD:C_0603"
+		(property "Footprint" "V2_Capacitor_SMD:C_1608"
 			(at 125.73 108.458 0)
 			(hide yes)
@@
 	)
 	(symbol
-		(lib_id "V2_Resistor:0603_100k")
+		(lib_id "V2_Resistor:1608_100k")
 		(at 177.8 93.98 0)
 		(unit 1)
@@
 			)
 		)
-		(property "Footprint" "V2_Resistor_SMD:R_0603"
+		(property "Footprint" "V2_Resistor_SMD:R_1608"
 			(at 177.8 109.728 0)
 			(hide yes)

Commit message: Refresh
Parts:
- renumbered C1404 to C1402, D1403 to D1401, R1407 to R1401
Changed lines of the file:
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@@
 	(title_block
 		(title "V2 sax")
-		(date "2026-04-23")
+		(date "2026-06-11")
 		(rev "2026-03-31")
 		(company "Versio Duo")
@@
 		(in_pos_files yes)
 		(dnp no)
-		(property "Reference" "C1404"
+		(property "Reference" "C1402"
 			(at 168.148 93.98 0)
 			(show_name no)
@@
 			(project "sax"
 				(path "/6c8448b4-b04d-47e1-934e-e40cbe27a7be/6178bc16-76cb-41ae-a61c-619a3590ea5a"
-					(reference "C1404")
+					(reference "C1402")
 					(unit 1)
 				)
@@
 		(dnp no)
 		(fields_autoplaced yes)
-		(property "Reference" "#PWR01407"
+		(property "Reference" "#PWR01402"
 			(at 125.73 100.33 0)
 			(hide yes)
@@
 			(project "sax"
 				(path "/6c8448b4-b04d-47e1-934e-e40cbe27a7be/6178bc16-76cb-41ae-a61c-619a3590ea5a"
-					(reference "#PWR01407")
+					(reference "#PWR01402")
 					(unit 1)
 				)
@@
 		(in_pos_files yes)
 		(dnp no)
-		(property "Reference" "#PWR01406"
+		(property "Reference" "#PWR01401"
 			(at 125.73 92.71 0)
 			(hide yes)
@@
 			(project "sax"
 				(path "/6c8448b4-b04d-47e1-934e-e40cbe27a7be/6178bc16-76cb-41ae-a61c-619a3590ea5a"
-					(reference "#PWR01406")
+					(reference "#PWR01401")
 					(unit 1)
 				)
@@
 		(in_pos_files yes)
 		(dnp no)
-		(property "Reference" "#PWR01412"
+		(property "Reference" "#PWR01403"
 			(at 152.4 86.36 0)
 			(hide yes)
@@
 			(project "sax"
 				(path "/6c8448b4-b04d-47e1-934e-e40cbe27a7be/6178bc16-76cb-41ae-a61c-619a3590ea5a"
-					(reference "#PWR01412")
+					(reference "#PWR01403")
 					(unit 1)
 				)
@@
 		(dnp no)
 		(fields_autoplaced yes)
-		(property "Reference" "#PWR01421"
+		(property "Reference" "#PWR01408"
 			(at 177.8 102.87 0)
 			(hide yes)
@@
 			(project "sax"
 				(path "/6c8448b4-b04d-47e1-934e-e40cbe27a7be/6178bc16-76cb-41ae-a61c-619a3590ea5a"
-					(reference "#PWR01421")
+					(reference "#PWR01408")
 					(unit 1)
 				)
@@
 		(dnp no)
 		(fields_autoplaced yes)
-		(property "Reference" "#PWR01420"
+		(property "Reference" "#PWR01407"
 			(at 165.1 102.87 0)
 			(hide yes)
@@
 			(project "sax"
 				(path "/6c8448b4-b04d-47e1-934e-e40cbe27a7be/6178bc16-76cb-41ae-a61c-619a3590ea5a"
-					(reference "#PWR01420")
+					(reference "#PWR01407")
 					(unit 1)
 				)
@@
 		(dnp no)
 		(fields_autoplaced yes)
-		(property "Reference" "#PWR01413"
+		(property "Reference" "#PWR01404"
 			(at 162.56 96.52 0)
 			(hide yes)
@@
 			(project "sax"
 				(path "/6c8448b4-b04d-47e1-934e-e40cbe27a7be/6178bc16-76cb-41ae-a61c-619a3590ea5a"
-					(reference "#PWR01413")
+					(reference "#PWR01404")
 					(unit 1)
 				)
@@
 		(in_pos_files yes)
 		(dnp no)
-		(property "Reference" "D1403"
+		(property "Reference" "D1401"
 			(at 150.876 120.65 0)
 			(show_name no)
@@
 			(project "sax"
 				(path "/6c8448b4-b04d-47e1-934e-e40cbe27a7be/6178bc16-76cb-41ae-a61c-619a3590ea5a"
-					(reference "D1403")
+					(reference "D1401")
 					(unit 1)
 				)
@@
 		(in_pos_files yes)
 		(dnp no)
-		(property "Reference" "#PWR01418"
+		(property "Reference" "#PWR01405"
 			(at 157.48 127 0)
 			(hide yes)
@@
 			(project "sax"
 				(path "/6c8448b4-b04d-47e1-934e-e40cbe27a7be/6178bc16-76cb-41ae-a61c-619a3590ea5a"
-					(reference "#PWR01418")
+					(reference "#PWR01405")
 					(unit 1)
 				)
@@
 		(in_pos_files yes)
 		(dnp no)
-		(property "Reference" "R1407"
+		(property "Reference" "R1401"
 			(at 185.42 93.9799 0)
 			(show_name no)
@@
 			(project "sax"
 				(path "/6c8448b4-b04d-47e1-934e-e40cbe27a7be/6178bc16-76cb-41ae-a61c-619a3590ea5a"
-					(reference "R1407")
+					(reference "R1401")
 					(unit 1)
 				)
@@
 		(in_pos_files yes)
 		(dnp no)
-		(property "Reference" "#PWR01419"
+		(property "Reference" "#PWR01406"
 			(at 167.64 132.08 0)
 			(hide yes)
@@
 			(project "sax"
 				(path "/6c8448b4-b04d-47e1-934e-e40cbe27a7be/6178bc16-76cb-41ae-a61c-619a3590ea5a"
-					(reference "#PWR01419")
+					(reference "#PWR01406")
 					(unit 1)
 				)
