File: hardware/sax/sax.kicad_pcb (KiCad board)
At the start: 4 copper layers, 80 x 34.5 mm, 103 parts, among them IC1401 MP3V5004GP, J101 Cortex, J102 DX07S016JA3, J1101 NE8FAH, J1301 2x05_Horizontal, SW101 SKSG, SW102 SKSG, U101 TPS78433QWDRBRQ1, U102 ATSAMD51J, U1101 THVD2442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

Commit message: Update
Connections:
- net /+VDDCORE renamed /+VCORE

Commit message: Update
Parts:
- renumbered C107 to C101, C110 to C102, C111 to C103, C101 to C104, C102 to C105, C103 to C106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
