File: hardware/sax/HallSensors.kicad_sch (KiCad schematic)
At the start: 2 parts, among them J1301 2x05_Horizontal

Commit message: Update
Parts:
- J1301: Rating (none) -> 1A
Changed lines of the file:
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@@
 	(title_block
 		(title "V2 sax")
-		(date "2026-04-10")
+		(date "2026-04-23")
 		(rev "2026-03-31")
 		(company "Versio Duo")
@@
 			)
 		)
+		(property "Rating" "1A"
+			(at 132.08 187.96 0)
+			(hide yes)
+			(show_name no)
+			(do_not_autoplace no)
+			(effects
+				(font
+					(size 1.27 1.27)
+				)
+			)
+		)
 		(pin "1"
 		)
@@
 		(in_pos_files yes)
 		(dnp no)
-		(property "Reference" "#PWR1304"
+		(property "Reference" "#PWR01302"
 			(at 134.62 162.56 0)
 			(hide yes)
@@
 			(project "sax"
 				(path "/6c8448b4-b04d-47e1-934e-e40cbe27a7be/986c2710-b6fb-48af-9291-0e7dc7b5abf9"
-					(reference "#PWR1304")
+					(reference "#PWR01302")
 					(unit 1)
 				)
@@
 		(in_pos_files yes)
 		(dnp no)
-		(property "Reference" "#PWR1302"
+		(property "Reference" "#PWR01304"
 			(at 167.64 166.37 0)
 			(hide yes)
@@
 			(project "sax"
 				(path "/6c8448b4-b04d-47e1-934e-e40cbe27a7be/986c2710-b6fb-48af-9291-0e7dc7b5abf9"
-					(reference "#PWR1302")
+					(reference "#PWR01304")
 					(unit 1)
 				)
@@
 		(in_pos_files yes)
 		(dnp no)
-		(property "Reference" "#PWR1303"
+		(property "Reference" "#PWR01301"
 			(at 119.38 162.56 0)
 			(hide yes)
@@
 			(project "sax"
 				(path "/6c8448b4-b04d-47e1-934e-e40cbe27a7be/986c2710-b6fb-48af-9291-0e7dc7b5abf9"
-					(reference "#PWR1303")
+					(reference "#PWR01301")
 					(unit 1)
 				)
@@
 		(in_pos_files yes)
 		(dnp no)
-		(property "Reference" "#PWR1301"
+		(property "Reference" "#PWR01303"
 			(at 167.64 156.21 0)
 			(hide yes)
@@
 			(project "sax"
 				(path "/6c8448b4-b04d-47e1-934e-e40cbe27a7be/986c2710-b6fb-48af-9291-0e7dc7b5abf9"
-					(reference "#PWR1301")
+					(reference "#PWR01303")
 					(unit 1)
 				)

Commit message: Refresh
Parts:
- TVS401: renamed from TVS1301; footprint V2_Diode_SMD:D_0603 -> V2_Diode_SMD:D_1608
- renumbered J1301 to J401
Changed lines of the file:
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@@
 	(title_block
 		(title "V2 sax")
-		(date "2026-04-23")
+		(date "2026-06-11")
 		(rev "2026-03-31")
 		(company "Versio Duo")
@@
 		(in_pos_files yes)
 		(dnp no)
-		(property "Reference" "J1301"
+		(property "Reference" "J401"
 			(at 133.35 144.78 0)
 			(show_name no)
@@
 			(project "sax"
 				(path "/6c8448b4-b04d-47e1-934e-e40cbe27a7be/986c2710-b6fb-48af-9291-0e7dc7b5abf9"
-					(reference "J1301")
+					(reference "J401")
 					(unit 1)
 				)
@@
 		(in_pos_files yes)
 		(dnp no)
-		(property "Reference" "#PWR01302"
+		(property "Reference" "#PWR0402"
 			(at 134.62 162.56 0)
 			(hide yes)
@@
 			(project "sax"
 				(path "/6c8448b4-b04d-47e1-934e-e40cbe27a7be/986c2710-b6fb-48af-9291-0e7dc7b5abf9"
-					(reference "#PWR01302")
+					(reference "#PWR0402")
 					(unit 1)
 				)
@@
 		(in_pos_files yes)
 		(dnp no)
-		(property "Reference" "TVS1301"
+		(property "Reference" "TVS401"
 			(at 174.752 154.94 90)
 			(show_name no)
@@
 			)
 		)
-		(property "Footprint" "V2_Diode_SMD:D_0603"
+		(property "Footprint" "V2_Diode_SMD:D_1608"
 			(at 173.355 156.21 0)
 			(hide yes)
@@
 			(project "sax"
 				(path "/6c8448b4-b04d-47e1-934e-e40cbe27a7be/986c2710-b6fb-48af-9291-0e7dc7b5abf9"
-					(reference "TVS1301")
+					(reference "TVS401")
 					(unit 1)
 				)
@@
 		(in_pos_files yes)
 		(dnp no)
-		(property "Reference" "#PWR01304"
+		(property "Reference" "#PWR0404"
 			(at 167.64 166.37 0)
 			(hide yes)
@@
 			(project "sax"
 				(path "/6c8448b4-b04d-47e1-934e-e40cbe27a7be/986c2710-b6fb-48af-9291-0e7dc7b5abf9"
-					(reference "#PWR01304")
+					(reference "#PWR0404")
 					(unit 1)
 				)
@@
 		(in_pos_files yes)
 		(dnp no)
-		(property "Reference" "#PWR01301"
+		(property "Reference" "#PWR0401"
 			(at 119.38 162.56 0)
 			(hide yes)
@@
 			(project "sax"
 				(path "/6c8448b4-b04d-47e1-934e-e40cbe27a7be/986c2710-b6fb-48af-9291-0e7dc7b5abf9"
-					(reference "#PWR01301")
+					(reference "#PWR0401")
 					(unit 1)
 				)
@@
 		(in_pos_files yes)
 		(dnp no)
-		(property "Reference" "#PWR01303"
+		(property "Reference" "#PWR0403"
 			(at 167.64 156.21 0)
 			(hide yes)
@@
 			(project "sax"
 				(path "/6c8448b4-b04d-47e1-934e-e40cbe27a7be/986c2710-b6fb-48af-9291-0e7dc7b5abf9"
-					(reference "#PWR01303")
+					(reference "#PWR0403")
 					(unit 1)
 				)
@@
 			(project "sax"
 				(path "/6c8448b4-b04d-47e1-934e-e40cbe27a7be/986c2710-b6fb-48af-9291-0e7dc7b5abf9"
-					(page "17")
+					(page "8")
 				)
 			)
@@
 			(project "sax"
 				(path "/6c8448b4-b04d-47e1-934e-e40cbe27a7be/986c2710-b6fb-48af-9291-0e7dc7b5abf9"
-					(page "14")
+					(page "5")
 				)
 			)
@@
 			(project "sax"
 				(path "/6c8448b4-b04d-47e1-934e-e40cbe27a7be/986c2710-b6fb-48af-9291-0e7dc7b5abf9"
-					(page "15")
+					(page "6")
 				)
 			)
@@
 			(project "sax"
 				(path "/6c8448b4-b04d-47e1-934e-e40cbe27a7be/986c2710-b6fb-48af-9291-0e7dc7b5abf9"
-					(page "21")
+					(page "12")
 				)
 			)
@@
 			(project "sax"
 				(path "/6c8448b4-b04d-47e1-934e-e40cbe27a7be/986c2710-b6fb-48af-9291-0e7dc7b5abf9"
-					(page "19")
+					(page "10")
 				)
 			)
@@
 			(project "sax"
 				(path "/6c8448b4-b04d-47e1-934e-e40cbe27a7be/986c2710-b6fb-48af-9291-0e7dc7b5abf9"
-					(page "16")
+					(page "7")
 				)
 			)
@@
 			(project "sax"
 				(path "/6c8448b4-b04d-47e1-934e-e40cbe27a7be/986c2710-b6fb-48af-9291-0e7dc7b5abf9"
-					(page "20")
+					(page "11")
 				)
 			)
@@
 			(project "sax"
 				(path "/6c8448b4-b04d-47e1-934e-e40cbe27a7be/986c2710-b6fb-48af-9291-0e7dc7b5abf9"
-					(page "18")
-				)
-			)
+					(page "9")
+				)
+			)
