File: hardware/sax/PowerSupply.kicad_sch (KiCad schematic)
At the start: 6 parts, among them U1201 TPSM33620S5QRDNRQ1

Commit message: Update
Parts:
- renumbered C1205 to C1203, C1203 to C1204, C1204 to C1205
Changed lines of the file:
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@@
 	(title_block
 		(title "V2 sax")
-		(date "2026-04-10")
+		(date "2026-04-23")
 		(rev "2026-03-31")
 		(company "Versio Duo")
@@
 		(in_pos_files yes)
 		(dnp no)
-		(property "Reference" "C1204"
+		(property "Reference" "C1205"
 			(at 198.12 96.52 0)
 			(show_name no)
@@
 			(project "sax"
 				(path "/6c8448b4-b04d-47e1-934e-e40cbe27a7be/095cddf1-6522-4d3b-885d-b21acd91d0c6"
-					(reference "C1204")
+					(reference "C1205")
 					(unit 1)
 				)
@@
 		(in_pos_files yes)
 		(dnp no)
-		(property "Reference" "#PWR1203"
+		(property "Reference" "#PWR01206"
 			(at 185.42 106.68 0)
 			(hide yes)
@@
 			(project "sax"
 				(path "/6c8448b4-b04d-47e1-934e-e40cbe27a7be/095cddf1-6522-4d3b-885d-b21acd91d0c6"
-					(reference "#PWR1203")
+					(reference "#PWR01206")
 					(unit 1)
 				)
@@
 		(in_pos_files yes)
 		(dnp no)
-		(property "Reference" "#PWR1204"
+		(property "Reference" "#PWR01207"
 			(at 195.58 106.68 0)
 			(hide yes)
@@
 			(project "sax"
 				(path "/6c8448b4-b04d-47e1-934e-e40cbe27a7be/095cddf1-6522-4d3b-885d-b21acd91d0c6"
-					(reference "#PWR1204")
+					(reference "#PWR01207")
 					(unit 1)
 				)
@@
 		(in_pos_files yes)
 		(dnp no)
-		(property "Reference" "#PWR1201"
+		(property "Reference" "#PWR01201"
 			(at 97.79 106.68 0)
 			(hide yes)
@@
 			(project "sax"
 				(path "/6c8448b4-b04d-47e1-934e-e40cbe27a7be/095cddf1-6522-4d3b-885d-b21acd91d0c6"
-					(reference "#PWR1201")
+					(reference "#PWR01201")
 					(unit 1)
 				)
@@
 		(in_pos_files yes)
 		(dnp no)
-		(property "Reference" "#PWR1202"
+		(property "Reference" "#PWR01202"
 			(at 109.22 106.68 0)
 			(hide yes)
@@
 			(project "sax"
 				(path "/6c8448b4-b04d-47e1-934e-e40cbe27a7be/095cddf1-6522-4d3b-885d-b21acd91d0c6"
-					(reference "#PWR1202")
+					(reference "#PWR01202")
 					(unit 1)
 				)
@@
 		(in_pos_files yes)
 		(dnp no)
-		(property "Reference" "C1205"
+		(property "Reference" "C1203"
 			(at 122.682 109.22 90)
 			(show_name no)
@@
 			(project "sax"
 				(path "/6c8448b4-b04d-47e1-934e-e40cbe27a7be/095cddf1-6522-4d3b-885d-b21acd91d0c6"
-					(reference "C1205")
+					(reference "C1203")
 					(unit 1)
 				)
@@
 		(in_pos_files yes)
 		(dnp no)
-		(property "Reference" "C1203"
+		(property "Reference" "C1204"
 			(at 187.96 96.52 0)
 			(show_name no)
@@
 			(project "sax"
 				(path "/6c8448b4-b04d-47e1-934e-e40cbe27a7be/095cddf1-6522-4d3b-885d-b21acd91d0c6"
-					(reference "C1203")
+					(reference "C1204")
 					(unit 1)
 				)
@@
 		(in_pos_files yes)
 		(dnp no)
-		(property "Reference" "#PWR1206"
+		(property "Reference" "#PWR01203"
 			(at 116.84 105.41 0)
 			(hide yes)
@@
 			(project "sax"
 				(path "/6c8448b4-b04d-47e1-934e-e40cbe27a7be/095cddf1-6522-4d3b-885d-b21acd91d0c6"
-					(reference "#PWR1206")
+					(reference "#PWR01203")
 					(unit 1)
 				)
@@
 		(in_pos_files yes)
 		(dnp no)
-		(property "Reference" "#PWR1208"
+		(property "Reference" "#PWR01204"
 			(at 129.54 110.49 0)
 			(hide yes)
@@
 			(project "sax"
 				(path "/6c8448b4-b04d-47e1-934e-e40cbe27a7be/095cddf1-6522-4d3b-885d-b21acd91d0c6"
-					(reference "#PWR1208")
+					(reference "#PWR01204")
 					(unit 1)
 				)
@@
 		(in_pos_files yes)
 		(dnp no)
-		(property "Reference" "#PWR1207"
+		(property "Reference" "#PWR01205"
 			(at 148.59 121.92 0)
 			(hide yes)
@@
 			(project "sax"
 				(path "/6c8448b4-b04d-47e1-934e-e40cbe27a7be/095cddf1-6522-4d3b-885d-b21acd91d0c6"
-					(reference "#PWR1207")
+					(reference "#PWR01205")
 					(unit 1)
 				)

Commit message: Good Bye Imperial
Parts:
- C1201: footprint V2_Capacitor_SMD:C_1210 -> V2_Capacitor_SMD:C_3225; symbol V2_Capacitor:1210_10u -> V2_Capacitor:3225_10u
- C1202: footprint V2_Capacitor_SMD:C_0603 -> V2_Capacitor_SMD:C_1608; symbol V2_Capacitor:0603_0u1 -> V2_Capacitor:1608_0u1
- C1203: footprint V2_Capacitor_SMD:C_0603 -> V2_Capacitor_SMD:C_1608; symbol V2_Capacitor:0603_1u -> V2_Capacitor:1608_1u
- C1204, C1205: footprint V2_Capacitor_SMD:C_1210 -> V2_Capacitor_SMD:C_3225; symbol V2_Capacitor:1210_22u -> V2_Capacitor:3225_22u
Changed lines of the file:
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@@
 	)
 	(symbol
-		(lib_id "V2_Capacitor:0603_0u1")
+		(lib_id "V2_Capacitor:1608_0u1")
 		(at 109.22 97.79 0)
 		(unit 1)
@@
 			)
 		)
-		(property "Footprint" "V2_Capacitor_SMD:C_0603"
+		(property "Footprint" "V2_Capacitor_SMD:C_1608"
 			(at 109.22 114.808 0)
 			(hide yes)
@@
 	)
 	(symbol
-		(lib_id "V2_Capacitor:1210_22u")
+		(lib_id "V2_Capacitor:3225_22u")
 		(at 195.58 97.79 0)
 		(unit 1)
@@
 			)
 		)
-		(property "Footprint" "V2_Capacitor_SMD:C_1210"
+		(property "Footprint" "V2_Capacitor_SMD:C_3225"
 			(at 195.58 114.808 0)
 			(hide yes)
@@
 	)
 	(symbol
-		(lib_id "V2_Capacitor:0603_1u")
+		(lib_id "V2_Capacitor:1608_1u")
 		(at 125.73 105.41 270)
 		(unit 1)
@@
 			)
 		)
-		(property "Footprint" "V2_Capacitor_SMD:C_0603"
+		(property "Footprint" "V2_Capacitor_SMD:C_1608"
 			(at 108.712 105.41 0)
 			(hide yes)
@@
 	)
 	(symbol
-		(lib_id "V2_Capacitor:1210_22u")
+		(lib_id "V2_Capacitor:3225_22u")
 		(at 185.42 97.79 0)
 		(unit 1)
@@
 			)
 		)
-		(property "Footprint" "V2_Capacitor_SMD:C_1210"
+		(property "Footprint" "V2_Capacitor_SMD:C_3225"
 			(at 185.42 114.808 0)
 			(hide yes)
@@
 	)
 	(symbol
-		(lib_id "V2_Capacitor:1210_10u")
+		(lib_id "V2_Capacitor:3225_10u")
 		(at 97.79 97.79 0)
 		(unit 1)
@@
 			)
 		)
-		(property "Footprint" "V2_Capacitor_SMD:C_1210"
+		(property "Footprint" "V2_Capacitor_SMD:C_3225"
 			(at 97.79 114.808 0)
 			(hide yes)

Commit message: Refresh
Parts:
- renumbered C1201 to C301, C1202 to C302, C1203 to C303, C1204 to C304, C1205 to C305, U1201 to U301
Changed lines of the file:
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@@
 	(title_block
 		(title "V2 sax")
-		(date "2026-04-23")
+		(date "2026-06-11")
 		(rev "2026-03-31")
 		(company "Versio Duo")
@@
 		(in_pos_files yes)
 		(dnp no)
-		(property "Reference" "U1201"
+		(property "Reference" "U301"
 			(at 141.986 87.63 0)
 			(show_name no)
@@
 			(project "sax"
 				(path "/6c8448b4-b04d-47e1-934e-e40cbe27a7be/095cddf1-6522-4d3b-885d-b21acd91d0c6"
-					(reference "U1201")
+					(reference "U301")
 					(unit 1)
 				)
@@
 		(in_pos_files yes)
 		(dnp no)
-		(property "Reference" "C1202"
+		(property "Reference" "C302"
 			(at 111.76 96.52 0)
 			(show_name no)
@@
 			(project "sax"
 				(path "/6c8448b4-b04d-47e1-934e-e40cbe27a7be/095cddf1-6522-4d3b-885d-b21acd91d0c6"
-					(reference "C1202")
+					(reference "C302")
 					(unit 1)
 				)
@@
 		(in_pos_files yes)
 		(dnp no)
-		(property "Reference" "C1205"
+		(property "Reference" "C305"
 			(at 198.12 96.52 0)
 			(show_name no)
@@
 			(project "sax"
 				(path "/6c8448b4-b04d-47e1-934e-e40cbe27a7be/095cddf1-6522-4d3b-885d-b21acd91d0c6"
-					(reference "C1205")
+					(reference "C305")
 					(unit 1)
 				)
@@
 		(in_pos_files yes)
 		(dnp no)
-		(property "Reference" "#PWR01206"
+		(property "Reference" "#PWR0306"
 			(at 185.42 106.68 0)
 			(hide yes)
@@
 			(project "sax"
 				(path "/6c8448b4-b04d-47e1-934e-e40cbe27a7be/095cddf1-6522-4d3b-885d-b21acd91d0c6"
-					(reference "#PWR01206")
+					(reference "#PWR0306")
 					(unit 1)
 				)
@@
 		(in_pos_files yes)
 		(dnp no)
-		(property "Reference" "#PWR01207"
+		(property "Reference" "#PWR0307"
 			(at 195.58 106.68 0)
 			(hide yes)
@@
 			(project "sax"
 				(path "/6c8448b4-b04d-47e1-934e-e40cbe27a7be/095cddf1-6522-4d3b-885d-b21acd91d0c6"
-					(reference "#PWR01207")
+					(reference "#PWR0307")
 					(unit 1)
 				)
@@
 		(in_pos_files yes)
 		(dnp no)
-		(property "Reference" "#PWR01201"
+		(property "Reference" "#PWR0301"
 			(at 97.79 106.68 0)
 			(hide yes)
@@
 			(project "sax"
 				(path "/6c8448b4-b04d-47e1-934e-e40cbe27a7be/095cddf1-6522-4d3b-885d-b21acd91d0c6"
-					(reference "#PWR01201")
+					(reference "#PWR0301")
 					(unit 1)
 				)
@@
 		(in_pos_files yes)
 		(dnp no)
-		(property "Reference" "#PWR01202"
+		(property "Reference" "#PWR0302"
 			(at 109.22 106.68 0)
 			(hide yes)
@@
 			(project "sax"
 				(path "/6c8448b4-b04d-47e1-934e-e40cbe27a7be/095cddf1-6522-4d3b-885d-b21acd91d0c6"
-					(reference "#PWR01202")
+					(reference "#PWR0302")
 					(unit 1)
 				)
@@
 		(in_pos_files yes)
 		(dnp no)
-		(property "Reference" "C1203"
+		(property "Reference" "C303"
 			(at 122.682 109.22 90)
 			(show_name no)
@@
 			(project "sax"
 				(path "/6c8448b4-b04d-47e1-934e-e40cbe27a7be/095cddf1-6522-4d3b-885d-b21acd91d0c6"
-					(reference "C1203")
+					(reference "C303")
 					(unit 1)
 				)
@@
 		(in_pos_files yes)
 		(dnp no)
-		(property "Reference" "C1204"
+		(property "Reference" "C304"
 			(at 187.96 96.52 0)
 			(show_name no)
@@
 			(project "sax"
 				(path "/6c8448b4-b04d-47e1-934e-e40cbe27a7be/095cddf1-6522-4d3b-885d-b21acd91d0c6"
-					(reference "C1204")
+					(reference "C304")
 					(unit 1)
 				)
@@
 		(in_pos_files yes)
 		(dnp no)
-		(property "Reference" "#PWR01203"
+		(property "Reference" "#PWR0303"
 			(at 116.84 105.41 0)
 			(hide yes)
@@
 			(project "sax"
 				(path "/6c8448b4-b04d-47e1-934e-e40cbe27a7be/095cddf1-6522-4d3b-885d-b21acd91d0c6"
-					(reference "#PWR01203")
+					(reference "#PWR0303")
 					(unit 1)
 				)
@@
 		(in_pos_files yes)
 		(dnp no)
-		(property "Reference" "#PWR01204"
+		(property "Reference" "#PWR0304"
 			(at 129.54 110.49 0)
 			(hide yes)
@@
 			(project "sax"
 				(path "/6c8448b4-b04d-47e1-934e-e40cbe27a7be/095cddf1-6522-4d3b-885d-b21acd91d0c6"
-					(reference "#PWR01204")
+					(reference "#PWR0304")
 					(unit 1)
 				)
@@
 		(in_pos_files yes)
 		(dnp no)
-		(property "Reference" "#PWR01205"
+		(property "Reference" "#PWR0305"
 			(at 148.59 121.92 0)
 			(hide yes)
@@
 			(project "sax"
 				(path "/6c8448b4-b04d-47e1-934e-e40cbe27a7be/095cddf1-6522-4d3b-885d-b21acd91d0c6"
-					(reference "#PWR01205")
+					(reference "#PWR0305")
 					(unit 1)
 				)
@@
 		(in_pos_files yes)
 		(dnp no)
-		(property "Reference" "C1201"
+		(property "Reference" "C301"
 			(at 100.33 96.52 0)
 			(show_name no)
@@
 			(project "sax"
 				(path "/6c8448b4-b04d-47e1-934e-e40cbe27a7be/095cddf1-6522-4d3b-885d-b21acd91d0c6"
-					(reference "C1201")
+					(reference "C301")
 					(unit 1)
 				)
