File: hardware/sax/sax.kicad_sch (KiCad schematic)
At the start: 36 parts, among them J101 Cortex, J102 DX07S016JA3, SW101 SKSG, SW102 SKSG, U101 TPS78433QWDRBRQ1, U102 ATSAMD51J, Y101 32k768

Commit message: Update
Parts:
- ESD101: Rating (none) -> 20kV
- U101: renamed from U102; Rating (none) -> Cortex-M4F
- renumbered C107 to C101, C110 to C102, C111 to C103, C101 to C104, C102 to C105, C103 to C106, C104 to C107, C105 to C108, C106 to C109, C108 to C110, C109 to C111, D105 to D101, D101 to D103, D103 to D104, D104 to D105, R104 to R101, R101 to R102, R102 to R103, R103 to R104, SW102 to SW101, SW101 to SW102, U101 to U102

Commit message: Good Bye Imperial
Parts:
- C101, C102: footprint V2_Capacitor_SMD:C_0603 -> V2_Capacitor_SMD:C_1608; symbol V2_Capacitor:0603_18p -> V2_Capacitor:1608_18p
- C103, C105, C106, C107, C108, C109: footprint V2_Capacitor_SMD:C_0603 -> V2_Capacitor_SMD:C_1608; symbol V2_Capacitor:0603_0u1 -> V2_Capacitor:1608_0u1
- C104: footprint V2_Capacitor_SMD:C_0603 -> V2_Capacitor_SMD:C_1608; symbol V2_Capacitor:0603_10u -> V2_Capacitor:1608_10u
- C110, C111: footprint V2_Capacitor_SMD:C_0805 -> V2_Capacitor_SMD:C_2012; symbol V2_Capacitor:0805_10u -> V2_Capacitor:2012_10u
- D102: symbol V2_LED:0603_Orange -> V2_LED:1608_Orange
- R101: footprint V2_Resistor_SMD:R_0603 -> V2_Resistor_SMD:R_1608; symbol V2_Resistor:0603_100k -> V2_Resistor:1608_100k
- R102: footprint V2_Resistor_SMD:R_0603 -> V2_Resistor_SMD:R_1608; symbol V2_Resistor:0603_330R -> V2_Resistor:1608_330R
- R103, R104: footprint V2_Resistor_SMD:R_0603 -> V2_Resistor_SMD:R_1608; symbol V2_Resistor:0603_5k1 -> V2_Resistor:1608_5k1
Changed lines of the file:
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@@
 	)
 	(symbol
-		(lib_id "V2_Capacitor:0603_0u1")
+		(lib_id "V2_Capacitor:1608_0u1")
 		(at 44.45 160.02 0)
 		(unit 1)
@@
 			)
 		)
-		(property "Footprint" "V2_Capacitor_SMD:C_0603"
+		(property "Footprint" "V2_Capacitor_SMD:C_1608"
 			(at 44.45 177.038 0)
 			(hide yes)
@@
 	)
 	(symbol
-		(lib_id "V2_Capacitor:0603_0u1")
+		(lib_id "V2_Capacitor:1608_0u1")
 		(at 88.9 26.67 0)
 		(unit 1)
@@
 			)
 		)
-		(property "Footprint" "V2_Capacitor_SMD:C_0603"
+		(property "Footprint" "V2_Capacitor_SMD:C_1608"
 			(at 88.9 43.688 0)
 			(hide yes)
@@
 	)
 	(symbol
-		(lib_id "V2_LED:0603_Orange")
+		(lib_id "V2_LED:1608_Orange")
 		(at 132.08 58.42 0)
 		(mirror y)
@@
 	)
 	(symbol
-		(lib_id "V2_Capacitor:0805_10u")
+		(lib_id "V2_Capacitor:2012_10u")
 		(at 198.12 39.37 0)
 		(unit 1)
@@
 			)
 		)
-		(property "Footprint" "V2_Capacitor_SMD:C_0805"
+		(property "Footprint" "V2_Capacitor_SMD:C_2012"
 			(at 198.12 56.388 0)
 			(hide yes)
@@
 	)
 	(symbol
-		(lib_id "V2_Capacitor:0603_18p")
+		(lib_id "V2_Capacitor:1608_18p")
 		(at 24.13 43.18 270)
 		(unit 1)
@@
 			)
 		)
-		(property "Footprint" "V2_Capacitor_SMD:C_0603"
+		(property "Footprint" "V2_Capacitor_SMD:C_1608"
 			(at 7.112 43.18 0)
 			(hide yes)
@@
 	)
 	(symbol
-		(lib_id "V2_Resistor:0603_5k1")
+		(lib_id "V2_Resistor:1608_5k1")
 		(at 207.01 88.9 90)
 		(unit 1)
@@
 			)
 		)
-		(property "Footprint" "V2_Resistor_SMD:R_0603"
+		(property "Footprint" "V2_Resistor_SMD:R_1608"
 			(at 222.758 88.9 0)
 			(hide yes)
@@
 	)
 	(symbol
-		(lib_id "V2_Capacitor:0805_10u")
+		(lib_id "V2_Capacitor:2012_10u")
 		(at 173.99 39.37 0)
 		(unit 1)
@@
 			)
 		)
-		(property "Footprint" "V2_Capacitor_SMD:C_0805"
+		(property "Footprint" "V2_Capacitor_SMD:C_2012"
 			(at 173.99 56.388 0)
 			(hide yes)
@@
 	)
 	(symbol
-		(lib_id "V2_Capacitor:0603_0u1")
+		(lib_id "V2_Capacitor:1608_0u1")
 		(at 119.38 26.67 0)
 		(unit 1)
@@
 			)
 		)
-		(property "Footprint" "V2_Capacitor_SMD:C_0603"
+		(property "Footprint" "V2_Capacitor_SMD:C_1608"
 			(at 119.38 43.688 0)
 			(hide yes)
@@
 	)
 	(symbol
-		(lib_id "V2_Resistor:0603_5k1")
+		(lib_id "V2_Resistor:1608_5k1")
 		(at 207.01 91.44 90)
 		(unit 1)
@@
 			)
 		)
-		(property "Footprint" "V2_Resistor_SMD:R_0603"
+		(property "Footprint" "V2_Resistor_SMD:R_1608"
 			(at 222.758 91.44 0)
 			(hide yes)
@@
 	)
 	(symbol
-		(lib_id "V2_Resistor:0603_100k")
+		(lib_id "V2_Resistor:1608_100k")
 		(at 50.8 120.65 90)
 		(unit 1)
@@
 			)
 		)
-		(property "Footprint" "V2_Resistor_SMD:R_0603"
+		(property "Footprint" "V2_Resistor_SMD:R_1608"
 			(at 66.548 120.65 0)
 			(hide yes)
@@
 	)
 	(symbol
-		(lib_id "V2_Capacitor:0603_18p")
+		(lib_id "V2_Capacitor:1608_18p")
 		(at 24.13 38.1 270)
 		(unit 1)
@@
 			)
 		)
-		(property "Footprint" "V2_Capacitor_SMD:C_0603"
+		(property "Footprint" "V2_Capacitor_SMD:C_1608"
 			(at 7.112 38.1 0)
 			(hide yes)
@@
 	)
 	(symbol
-		(lib_id "V2_Resistor:0603_330R")
+		(lib_id "V2_Resistor:1608_330R")
 		(at 139.7 58.42 90)
 		(unit 1)
@@
 			)
 		)
-		(property "Footprint" "V2_Resistor_SMD:R_0603"
+		(property "Footprint" "V2_Resistor_SMD:R_1608"
 			(at 155.448 58.42 0)
 			(hide yes)
@@
 	)
 	(symbol
-		(lib_id "V2_Capacitor:0603_0u1")
+		(lib_id "V2_Capacitor:1608_0u1")
 		(at 99.06 26.67 0)
 		(unit 1)
@@
 			)
 		)
-		(property "Footprint" "V2_Capacitor_SMD:C_0603"
+		(property "Footprint" "V2_Capacitor_SMD:C_1608"
 			(at 99.06 43.688 0)
 			(hide yes)
@@
 	)
 	(symbol
-		(lib_id "V2_Capacitor:0603_0u1")
+		(lib_id "V2_Capacitor:1608_0u1")
 		(at 78.74 26.67 0)
 		(unit 1)
@@
 			)
 		)
-		(property "Footprint" "V2_Capacitor_SMD:C_0603"
+		(property "Footprint" "V2_Capacitor_SMD:C_1608"
 			(at 78.74 43.688 0)
 			(hide yes)
@@
 	)
 	(symbol
-		(lib_id "V2_Capacitor:0603_0u1")
+		(lib_id "V2_Capacitor:1608_0u1")
 		(at 109.22 26.67 0)
 		(unit 1)
@@
 			)
 		)
-		(property "Footprint" "V2_Capacitor_SMD:C_0603"
+		(property "Footprint" "V2_Capacitor_SMD:C_1608"
 			(at 109.22 43.688 0)
 			(hide yes)
@@
 	)
 	(symbol
-		(lib_id "V2_Capacitor:0603_10u")
+		(lib_id "V2_Capacitor:1608_10u")
 		(at 57.15 26.67 0)
 		(unit 1)
@@
 			)
 		)
-		(property "Footprint" "V2_Capacitor_SMD:C_0603"
+		(property "Footprint" "V2_Capacitor_SMD:C_1608"
 			(at 57.15 43.688 0)
 			(hide yes)

Commit message: Refresh
Parts:
- D102: footprint V2_LED:LED_0603 -> V2_LED:LED_1608
- INFO102: value Layer_Numbers -> Layer_Numbers-4; footprint V2_Production:Layer_Numbers -> V2_Production:Layer_Numbers-4; symbol V2_Production:Layer_Numbers -> V2_Production:Layer_Numbers-4
Other:
- moved on the sheet: ICON101, INFO101, INFO102
Changed lines of the file:
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@@
 	(title_block
 		(title "V2 sax")
-		(date "2026-04-23")
+		(date "2026-06-11")
 		(rev "2026-03-31")
 		(company "Versio Duo")
@@
 	)
 	(symbol
-		(lib_id "V2_Production:Layer_Numbers")
-		(at 213.36 166.37 0)
+		(lib_id "V2_Production:Layer_Numbers-4")
+		(at 208.28 167.64 0)
 		(unit 1)
 		(body_style 1)
@@
 		(dnp no)
 		(property "Reference" "INFO102"
-			(at 220.218 166.37 0)
+			(at 215.138 167.64 0)
 			(show_name no)
 			(do_not_autoplace no)
@@
 			)
 		)
-		(property "Value" "Layer_Numbers"
-			(at 208.28 162.5599 0)
+		(property "Value" "Layer_Numbers-4"
+			(at 203.2 163.8299 0)
 			(hide yes)
 			(show_name no)
@@
 			)
 		)
-		(property "Footprint" "V2_Production:Layer_Numbers"
-			(at 213.36 172.72 0)
+		(property "Footprint" "V2_Production:Layer_Numbers-4"
+			(at 208.28 173.99 0)
 			(hide yes)
 			(show_name no)
@@
 		)
 		(property "Datasheet" ""
-			(at 213.36 168.91 0)
+			(at 208.28 170.18 0)
 			(hide yes)
 			(show_name no)
@@
 		)
 		(property "Description" ""
-			(at 213.36 166.37 0)
+			(at 208.28 167.64 0)
 			(hide yes)
 			(show_name no)
@@
 			)
 		)
-		(property "Footprint" "V2_LED:LED_0603"
+		(property "Footprint" "V2_LED:LED_1608"
 			(at 132.08 58.42 90)
 			(hide yes)
@@
 	(symbol
 		(lib_id "V2_Production:Revision")
-		(at 213.36 160.02 0)
+		(at 210.82 160.02 0)
 		(unit 1)
 		(body_style 1)
@@
 		(dnp no)
 		(property "Reference" "INFO101"
-			(at 224.028 160.02 0)
+			(at 221.488 160.02 0)
 			(show_name no)
 			(do_not_autoplace no)
@@
 		)
 		(property "Value" ""
-			(at 213.36 162.56 0)
+			(at 210.82 162.56 0)
 			(hide yes)
 			(show_name no)
@@
 		)
 		(property "Footprint" "V2_Production:Revision"
-			(at 213.36 165.1 0)
+			(at 210.82 165.1 0)
 			(hide yes)
 			(show_name no)
@@
 		)
 		(property "Datasheet" ""
-			(at 213.36 160.02 0)
+			(at 210.82 160.02 0)
 			(hide yes)
 			(show_name no)
@@
 		)
 		(property "Description" ""
-			(at 213.36 160.02 0)
+			(at 210.82 160.02 0)
 			(hide yes)
 			(show_name no)
@@
 	(symbol
 		(lib_id "V2_Artwork:V2-logo")
-		(at 212.09 151.13 0)
+		(at 209.55 151.13 0)
 		(unit 1)
 		(body_style 1)
@@
 		(dnp no)
 		(property "Reference" "ICON101"
-			(at 215.9 151.13 0)
+			(at 213.36 151.13 0)
 			(show_name no)
 			(do_not_autoplace no)
@@
 		)
 		(property "Value" "V2-logo"
-			(at 208.28 146.05 0)
+			(at 205.74 146.05 0)
 			(hide yes)
 			(show_name no)
@@
 		)
 		(property "Footprint" "V2_Artwork:Logo_Small"
-			(at 212.09 158.75 0)
+			(at 209.55 158.75 0)
 			(hide yes)
 			(show_name no)
@@
 		)
 		(property "Datasheet" ""
-			(at 212.09 151.13 0)
+			(at 209.55 151.13 0)
 			(hide yes)
 			(show_name no)
@@
 		)
 		(property "Description" ""
-			(at 212.09 151.13 0)
+			(at 209.55 151.13 0)
 			(hide yes)
 			(show_name no)
@@
 			(project "sax"
 				(path "/6c8448b4-b04d-47e1-934e-e40cbe27a7be"
-					(page "12")
+					(page "3")
 				)
 			)
@@
 			(project "sax"
 				(path "/6c8448b4-b04d-47e1-934e-e40cbe27a7be"
-					(page "13")
+					(page "4")
 				)
 			)
@@
 			(project "sax"
 				(path "/6c8448b4-b04d-47e1-934e-e40cbe27a7be"
-					(page "11")
+					(page "2")
 				)
 			)
@@
 			(project "sax"
 				(path "/6c8448b4-b04d-47e1-934e-e40cbe27a7be"
-					(page "14")
+					(page "13")
 				)
 			)
